File: mclk.kicad_sch (KiCad schematic)
At the start: 11 parts, among them J13 Conn_Coaxial, U6 74LVC1G17, U7 74LVC1G17

Commit message: redoing file add
Parts:
- renumbered C22 to C26, C23 to C27, C24 to C28, R39 to R35, R40 to R36, R41 to R37, R42 to R38
Changed lines of the file:
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@@
 		(dnp no)
 		(fields_autoplaced yes)
-		(property "Reference" "R39"
+		(property "Reference" "R35"
 			(at 114.3 67.7133 90)
 			(effects
@@
 			(project "pcm3168a_euro1"
 				(path "/afe1fbe1-30b6-4eb7-94cf-5d2700d51271/c547ec39-eaea-4f85-aadd-87956f9fb5f2"
-					(reference "R39")
+					(reference "R35")
 					(unit 1)
 				)
@@
 		(dnp yes)
 		(fields_autoplaced yes)
-		(property "Reference" "R40"
+		(property "Reference" "R36"
 			(at 122.1486 78.7978 0)
 			(effects
@@
 			(project "pcm3168a_euro1"
 				(path "/afe1fbe1-30b6-4eb7-94cf-5d2700d51271/c547ec39-eaea-4f85-aadd-87956f9fb5f2"
-					(reference "R40")
+					(reference "R36")
 					(unit 1)
 				)
@@
 		(dnp no)
 		(fields_autoplaced yes)
-		(property "Reference" "C24"
+		(property "Reference" "C28"
 			(at 161.671 105.4678 0)
 			(effects
@@
 			(project "pcm3168a_euro1"
 				(path "/afe1fbe1-30b6-4eb7-94cf-5d2700d51271/c547ec39-eaea-4f85-aadd-87956f9fb5f2"
-					(reference "C24")
+					(reference "C28")
 					(unit 1)
 				)
@@
 		(dnp no)
 		(fields_autoplaced yes)
-		(property "Reference" "R41"
+		(property "Reference" "R37"
 			(at 176.53 67.7133 90)
 			(effects
@@
 			(project "pcm3168a_euro1"
 				(path "/afe1fbe1-30b6-4eb7-94cf-5d2700d51271/c547ec39-eaea-4f85-aadd-87956f9fb5f2"
-					(reference "R41")
+					(reference "R37")
 					(unit 1)
 				)
@@
 		(dnp no)
 		(fields_autoplaced yes)
-		(property "Reference" "#PWR056"
+		(property "Reference" "#PWR060"
 			(at 158.75 68.58 0)
 			(effects
@@
 			(project "pcm3168a_euro1"
 				(path "/afe1fbe1-30b6-4eb7-94cf-5d2700d51271/c547ec39-eaea-4f85-aadd-87956f9fb5f2"
-					(reference "#PWR056")
+					(reference "#PWR060")
 					(unit 1)
 				)
@@
 		(dnp no)
 		(fields_autoplaced yes)
-		(property "Reference" "C23"
+		(property "Reference" "C27"
 			(at 161.671 57.2078 0)
 			(effects
@@
 			(project "pcm3168a_euro1"
 				(path "/afe1fbe1-30b6-4eb7-94cf-5d2700d51271/c547ec39-eaea-4f85-aadd-87956f9fb5f2"
-					(reference "C23")
+					(reference "C27")
 					(unit 1)
 				)
@@
 		(dnp no)
 		(fields_autoplaced yes)
-		(property "Reference" "#PWR054"
+		(property "Reference" "#PWR058"
 			(at 152.4 105.41 0)
 			(effects
@@
 			(project "pcm3168a_euro1"
 				(path "/afe1fbe1-30b6-4eb7-94cf-5d2700d51271/c547ec39-eaea-4f85-aadd-87956f9fb5f2"
-					(reference "#PWR054")
+					(reference "#PWR058")
 					(unit 1)
 				)
@@
 		(dnp no)
 		(fields_autoplaced yes)
-		(property "Reference" "R42"
+		(property "Reference" "R38"
 			(at 176.53 115.9733 90)
 			(effects
@@
 			(project "pcm3168a_euro1"
 				(path "/afe1fbe1-30b6-4eb7-94cf-5d2700d51271/c547ec39-eaea-4f85-aadd-87956f9fb5f2"
-					(reference "R42")
+					(reference "R38")
 					(unit 1)
 				)
@@
 		(dnp no)
 		(fields_autoplaced yes)
-		(property "Reference" "#PWR055"
+		(property "Reference" "#PWR059"
 			(at 152.4 143.51 0)
 			(effects
@@
 			(project "pcm3168a_euro1"
 				(path "/afe1fbe1-30b6-4eb7-94cf-5d2700d51271/c547ec39-eaea-4f85-aadd-87956f9fb5f2"
-					(reference "#PWR055")
+					(reference "#PWR059")
 					(unit 1)
 				)
@@
 		(dnp no)
 		(fields_autoplaced yes)
-		(property "Reference" "#PWR053"
+		(property "Reference" "#PWR057"
 			(at 152.4 95.25 0)
 			(effects
@@
 			(project "pcm3168a_euro1"
 				(path "/afe1fbe1-30b6-4eb7-94cf-5d2700d51271/c547ec39-eaea-4f85-aadd-87956f9fb5f2"
-					(reference "#PWR053")
+					(reference "#PWR057")
 					(unit 1)
 				)
@@
 		(dnp no)
 		(fields_autoplaced yes)
-		(property "Reference" "#PWR051"
+		(property "Reference" "#PWR055"
 			(at 100.33 93.98 0)
 			(effects
@@
 			(project "pcm3168a_euro1"
 				(path "/afe1fbe1-30b6-4eb7-94cf-5d2700d51271/c547ec39-eaea-4f85-aadd-87956f9fb5f2"
-					(reference "#PWR051")
+					(reference "#PWR055")
 					(unit 1)
 				)
@@
 		(dnp no)
 		(fields_autoplaced yes)
-		(property "Reference" "#PWR057"
+		(property "Reference" "#PWR061"
 			(at 158.75 116.84 0)
 			(effects
@@
 			(project "pcm3168a_euro1"
 				(path "/afe1fbe1-30b6-4eb7-94cf-5d2700d51271/c547ec39-eaea-4f85-aadd-87956f9fb5f2"
-					(reference "#PWR057")
+					(reference "#PWR061")
 					(unit 1)
 				)
@@
 		(dnp no)
 		(fields_autoplaced yes)
-		(property "Reference" "#PWR052"
+		(property "Reference" "#PWR056"
 			(at 152.4 57.15 0)
 			(effects
@@
 			(project "pcm3168a_euro1"
 				(path "/afe1fbe1-30b6-4eb7-94cf-5d2700d51271/c547ec39-eaea-4f85-aadd-87956f9fb5f2"
-					(reference "#PWR052")
+					(reference "#PWR056")
 					(unit 1)
 				)
@@
 		(dnp yes)
 		(fields_autoplaced yes)
-		(property "Reference" "C22"
+		(property "Reference" "C26"
 			(at 135.6741 78.8041 0)
 			(effects
@@
 			(project "pcm3168a_euro1"
 				(path "/afe1fbe1-30b6-4eb7-94cf-5d2700d51271/c547ec39-eaea-4f85-aadd-87956f9fb5f2"
-					(reference "C22")
-					(unit 1)
-				)
+					(reference "C26")
+					(unit 1)
+				)
