File: pcm3168a_euro1.kicad_pcb (KiCad board)
At the start: 2 copper layers, 160 parts, among them J1 Conn_02x04_Odd_Even, J10 Conn_Coaxial, J11 Conn_Coaxial, J12 Conn_Coaxial, J13 Conn_Coaxial, J14 Conn_Coaxial, J15 Conn_Coaxial, J16 Conn_Coaxial, J17 Conn_02x08_Odd_Even, J18 Conn_Coaxial, J2 Conn_02x04_Odd_Even, J3 Conn_02x04_Odd_Even, J4 Conn_02x04_Odd_Even, J5 Conn_02x04_Odd_Even, J6 Conn_Coaxial, J7 Conn_Coaxial, J8 Conn_01x02_Pin, J9 Conn_Coaxial, U1 PCM3168APAPR, U10 74LVC1G17, U11 TLV1117-33, U12 OPA1637, U2 74LVC1G17, U3 74LVC1G17, U4 74LVC1G17, U5 74LVC1G17, U6 74LVC1G17, U7 74LVC1G17, U8 74LVC1G17, U9 74LVC1G17, Y1 SG-210STF 24.5760ML0

Commit message: redoing file add
Parts:
- added C35: C_Polarized_Small, Capacitor_THT:CP_Radial_D8.0mm_P3.50mm, F.Cu at (123.3, 118.6)
- added C36: C_Polarized_Small, Capacitor_THT:CP_Radial_D8.0mm_P3.50mm, F.Cu at (132.1, 118.6)
- added C37: 6.8n, Capacitor_SMD:C_0603_1608Metric, F.Cu at (127.8, 111.7)
- added C38: 1n, Capacitor_SMD:C_0603_1608Metric, F.Cu at (123.8, 109.4)
- added C39: 1n, Capacitor_SMD:C_0603_1608Metric, F.Cu at (131.8, 109.5)
- added C40: 100nF, Capacitor_SMD:C_0603_1608Metric, F.Cu at (127.8, 101.6)
- added C41: 39n, Capacitor_SMD:C_0603_1608Metric, F.Cu at (127.9, 99.8)
- added C71: 100nF, Capacitor_SMD:C_0603_1608Metric, F.Cu at (110.0, 101.6)
- added C73: C_Polarized_Small, Capacitor_THT:CP_Radial_D8.0mm_P3.50mm, F.Cu at (141.2, 118.6)
- added C74: C_Polarized_Small, Capacitor_THT:CP_Radial_D8.0mm_P3.50mm, F.Cu at (150.0, 118.7)
- added C75: 6.8n, Capacitor_SMD:C_0603_1608Metric, F.Cu at (145.7, 111.8)
- added C76: 1n, Capacitor_SMD:C_0603_1608Metric, F.Cu at (141.7, 109.5)
- added C77: 1n, Capacitor_SMD:C_0603_1608Metric, F.Cu at (149.7, 109.5)
- added C78: 100nF, Capacitor_SMD:C_0603_1608Metric, F.Cu at (145.7, 101.7)
- added C79: 39n, Capacitor_SMD:C_0603_1608Metric, F.Cu at (145.8, 99.8)
- added C80: C_Polarized_Small, Capacitor_THT:CP_Radial_D8.0mm_P3.50mm, F.Cu at (158.9, 118.8)
- added C81: C_Polarized_Small, Capacitor_THT:CP_Radial_D8.0mm_P3.50mm, F.Cu at (167.8, 118.8)
- added C82: 6.8n, Capacitor_SMD:C_0603_1608Metric, F.Cu at (163.5, 111.9)
- added C83: 1n, Capacitor_SMD:C_0603_1608Metric, F.Cu at (159.5, 109.7)
- added C84: 1n, Capacitor_SMD:C_0603_1608Metric, F.Cu at (167.4, 109.7)
- added C85: 100nF, Capacitor_SMD:C_0603_1608Metric, F.Cu at (163.4, 101.9)
- added C86: 39n, Capacitor_SMD:C_0603_1608Metric, F.Cu at (163.5, 100.0)
- added J17: ACJS-MV35-3, pcm3168a_euro1:Amphenol_ACJS, F.Cu at (127.7, 133.3)
- added J20: ACJS-MV35-3, pcm3168a_euro1:Amphenol_ACJS, F.Cu at (109.9, 133.3)
- added J21: ACJS-MV35-3, pcm3168a_euro1:Amphenol_ACJS, F.Cu at (145.6, 133.4)
- added J22: ACJS-MV35-3, pcm3168a_euro1:Amphenol_ACJS, F.Cu at (163.3, 133.6)
- added R48: 1.1k, Resistor_SMD:R_0603_1608Metric, F.Cu at (127.1, 114.0)
- added R49: 1.1k, Resistor_SMD:R_0603_1608Metric, F.Cu at (128.7, 114.0)
- added R50: 1.1k, Resistor_SMD:R_0603_1608Metric, F.Cu at (125.4, 109.4)
- added R51: 1.1k, Resistor_SMD:R_0603_1608Metric, F.Cu at (130.2, 109.5)
- added R52: 560, Resistor_SMD:R_0603_1608Metric, F.Cu at (127.0, 109.4)
- added R53: 560, Resistor_SMD:R_0603_1608Metric, F.Cu at (128.7, 109.4)
- added R54: 47, Resistor_SMD:R_0603_1608Metric, F.Cu at (125.4, 100.9)
- added R55: 47, Resistor_SMD:R_0603_1608Metric, F.Cu at (130.3, 100.9)
- added R66: 1.1k, Resistor_SMD:R_0603_1608Metric, F.Cu at (145.0, 114.1)
- added R67: 1.1k, Resistor_SMD:R_0603_1608Metric, F.Cu at (146.6, 114.1)
- added R68: 1.1k, Resistor_SMD:R_0603_1608Metric, F.Cu at (143.3, 109.5)
- added R69: 1.1k, Resistor_SMD:R_0603_1608Metric, F.Cu at (148.1, 109.5)
- added R70: 560, Resistor_SMD:R_0603_1608Metric, F.Cu at (144.9, 109.5)
- added R71: 560, Resistor_SMD:R_0603_1608Metric, F.Cu at (146.6, 109.5)
- added R72: 47, Resistor_SMD:R_0603_1608Metric, F.Cu at (143.3, 101.0)
- added R73: 47, Resistor_SMD:R_0603_1608Metric, F.Cu at (148.2, 100.9)
- added R74: 1.1k, Resistor_SMD:R_0603_1608Metric, F.Cu at (162.7, 114.2)
- added R75: 1.1k, Resistor_SMD:R_0603_1608Metric, F.Cu at (164.3, 114.2)
- added R76: 1.1k, Resistor_SMD:R_0603_1608Metric, F.Cu at (161.1, 109.6)
- added R77: 1.1k, Resistor_SMD:R_0603_1608Metric, F.Cu at (165.9, 109.7)
- added R78: 560, Resistor_SMD:R_0603_1608Metric, F.Cu at (162.6, 109.6)
- added R79: 560, Resistor_SMD:R_0603_1608Metric, F.Cu at (164.3, 109.7)
- added R80: 47, Resistor_SMD:R_0603_1608Metric, F.Cu at (161.0, 101.1)
- added R81: 47, Resistor_SMD:R_0603_1608Metric, F.Cu at (166.0, 101.1)
- added U11: OPA1637, Package_SO:SOIC-8_3.9x4.9mm_P1.27mm, F.Cu at (127.9, 105.2)
- added U14: OPA1637, Package_SO:SOIC-8_3.9x4.9mm_P1.27mm, F.Cu at (145.8, 105.2)
- added U15: OPA1637, Package_SO:SOIC-8_3.9x4.9mm_P1.27mm, F.Cu at (163.5, 105.4)
- moved J1 190.9 mm to (197.5, 84.4)
- moved J2 190.9 mm to (185.1, 84.4)
- moved J3 190.9 mm to (191.2, 84.4)
- moved J4 190.9 mm to (220.3, 84.1)
- moved J5 190.9 mm to (204.2, 84.4)
- moved J7 190.9 mm to (213.4, 87.9)
- moved R1 190.9 mm to (201.5, 85.6)
- moved R10 190.9 mm to (208.4, 90.8)
- moved R4 190.9 mm to (201.5, 90.7)
- moved R5 190.9 mm to (189.3, 90.7)
- moved R6 190.9 mm to (195.5, 90.8)
- moved R7 190.9 mm to (224.5, 85.4)
- moved R8 190.9 mm to (208.4, 85.8)
- moved R9 190.9 mm to (224.5, 90.4)
- moved J6 190.9 mm to (229.5, 87.9)
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- renumbered C201 to C1, C7 to C10, C61 to C11, C8 to C12, C9 to C13, C10 to C14, C11 to C15, C12 to C16, C13 to C17, C14 to C18, C15 to C19, C1 to C2, C16 to C20, C17 to C21, C18 to C22, C19 to C23, C20 to C24, C21 to C25, C22 to C26, C23 to C27, C24 to C28, C25 to C29, C2 to C3, C26 to C30, C27 to C31, C28 to C32, C29 to C33, C30 to C34, C3 to C4, C31 to C42, C32 to C43, C33 to C44, C34 to C45, C35 to C46, C36 to C47, C37 to C48, C38 to C49, C4 to C5, C39 to C50, C40 to C51, C41 to C52, C42 to C53, C43 to C54, C44 to C55, C45 to C56, C46 to C57, C47 to C58, C48 to C59, C5 to C6, C49 to C60, C50 to C61, C51 to C62, C52 to C63, C53 to C64, C54 to C65, C55 to C66, C56 to C67, C57 to C68, C58 to C69, C202 to C7, C59 to C70, C60 to C72, C200 to C8, C6 to C9, J17 to J18, J18 to J19, R23 to R19, R24 to R20, R25 to R21, R26 to R22, R27 to R23, R28 to R24, R29 to R25, R30 to R26, R31 to R27, R32 to R28, R33 to R29, R34 to R30, R35 to R31, R36 to R32, R37 to R33, R38 to R34, R39 to R35, R40 to R36, R41 to R37, R42 to R38, R43 to R39, R44 to R40, R45 to R41, R46 to R42, R47 to R43, R48 to R44, R49 to R45, R50 to R46, R51 to R47, R52 to R56, R53 to R57, R54 to R58, R55 to R59, R56 to R60, R57 to R61, R58 to R62, R59 to R63, R60 to R64, R61 to R65, U11 to U12, U12 to U13
Connections:
- C14 pad 1: Net-(U1-VCOMAD) -> VCOMAD
- C66 pad 2: unconnected-(C55-Pad2) -> Net-(J20-Pin_4)
- C67 pad 2: unconnected-(C56-Pad2) -> Net-(J20-Pin_3)
- C72 pad 1: Net-(C60-Pad1) -> /VIN1-
- C72 pad 2: Net-(C60-Pad2) -> /VIN1+
- R64 pad 1: Net-(C60-Pad1) -> /VIN1-
- R65 pad 2: Net-(C60-Pad2) -> /VIN1+
- U1 pad 1: Net-(U1-VCOMAD) -> VCOMAD
- U1 pad 51: unconnected-(U1-VIN1--Pad51) -> /VIN1-
- U1 pad 52: unconnected-(U1-VIN1+-Pad52) -> /VIN1+
- U1 pad 53: unconnected-(U1-VIN2--Pad53) -> /VIN2-
- U1 pad 54: unconnected-(U1-VIN2+-Pad54) -> /VIN2+
- U1 pad 55: unconnected-(U1-VIN3--Pad55) -> /VIN3-
- U1 pad 56: unconnected-(U1-VIN3+-Pad56) -> /VIN3+
- U1 pad 57: unconnected-(U1-VIN4--Pad57) -> /VIN4-
- U1 pad 58: unconnected-(U1-VIN4+-Pad58) -> /VIN4+
- U1 pad 61: unconnected-(U1-VIN5--Pad61) -> /VIN5-
- U1 pad 62: unconnected-(U1-VIN5+-Pad62) -> /VIN5+
- U1 pad 63: unconnected-(U1-VIN6--Pad63) -> /VIN6-
- U1 pad 64: unconnected-(U1-VIN6+-Pad64) -> /VIN6+
- U13 pad 2: /amp/VOCM -> VCOMAD
- U13 pad 3: unconnected-(U12-V+-Pad3) -> +5V
- U13 pad 6: unconnected-(U12-V--Pad6) -> GND
Routing:
- net VCOMAD: track 0.00 -> 100.6 mm, vias 0 -> 7
- net /dout1/IN: track 0.00 -> 83.7 mm, vias 0 -> 2
- net /LRCK: track 4.67 -> 67.9 mm, vias 0 -> 2
- net /BCK: track 2.14 -> 58.8 mm, vias 0 -> 2
- net /SCKI: track 1.68 -> 56.3 mm
- net /din1/OUT: track 0.00 -> 49.1 mm
- net /mclk/OUT1: track 0.00 -> 49.0 mm
- net /VIN4+: track 0.00 -> 38.8 mm
- net /VIN4-: track 0.00 -> 38.4 mm
- net /VIN1-: track 0.00 -> 35.7 mm
- net /VIN1+: track 0.00 -> 35.7 mm
- net Net-(J20-Pin_4): track 0.00 -> 25.4 mm
- net Net-(J17-Pin_4): track 0.00 -> 25.4 mm
- net Net-(J22-Pin_4): track 0.00 -> 25.4 mm
- net Net-(J21-Pin_4): track 0.00 -> 25.4 mm
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Other:
- board outline added: 196 x 128.4 mm

Commit message: WIP layout
Parts:
- removed C28: 100nF, Capacitor_SMD:C_0603_1608Metric
- removed C51, C52, C57, C58, C66: C_Polarized_Small, Capacitor_THT:CP_Radial_D8.0mm_P3.50mm
- removed C53, C54, C55, C56, C60, C61, C63, C64: C_Small, Capacitor_SMD:C_0603_1608Metric
- removed C69: 1n, Capacitor_SMD:C_0603_1608Metric
- removed D3, D4: D_Zener_Small, Diode_SMD:D_SOD-123F
- removed J16, J6, J7: Conn_Coaxial, Connector_Coaxial:SMA_Amphenol_901-144_Vertical
- removed J2, J3, J4, J5: Conn_02x04_Odd_Even, Connector_PinHeader_2.54mm:PinHeader_2x04_P2.54mm_Vertical
- removed J20: ACJS-MV35-3, pcm3168a_euro1:Amphenol_ACJS
- removed L3, L4: L_Ferrite_Small, Inductor_SMD:L_0603_1608Metric
- removed R10, R3, R4, R5, R6, R7, R8, R9: 220k 5%, Resistor_SMD:R_0603_1608Metric
- removed R12, R15, R17, R18, R45: 0, Resistor_SMD:R_0603_1608Metric
- removed R46: R_Small, Resistor_SMD:R_0603_1608Metric
- removed R47: 22, Resistor_SMD:R_0603_1608Metric
- removed U10, U7: 74LVC1G17, Package_TO_SOT_SMD:SOT-23-5
- added C100: 39n, Capacitor_SMD:C_0603_1608Metric, F.Cu at (160.4, 142.6)
- added C101: 100nF, Capacitor_SMD:C_0603_1608Metric, F.Cu at (169.1, 142.5)
- added C102: C_Polarized_Small, Capacitor_THT:CP_Radial_D8.0mm_P3.50mm, F.Cu at (175.6, 138.1)
- added C103: C_Polarized_Small, Capacitor_THT:CP_Radial_D8.0mm_P3.50mm, F.Cu at (175.7, 147.3)
- added C104: 6.8n, Capacitor_SMD:C_0603_1608Metric, F.Cu at (149.1, 160.9)
- added C105: 1n, Capacitor_SMD:C_0603_1608Metric, F.Cu at (151.3, 157.2)
- added C106: 1n, Capacitor_SMD:C_0603_1608Metric, F.Cu at (151.3, 164.7)
- added C107: 100nF, Capacitor_SMD:C_0603_1608Metric, F.Cu at (159.0, 161.1)
- added C108: 39n, Capacitor_SMD:C_0603_1608Metric, F.Cu at (160.4, 161.0)
- added C109: 100nF, Capacitor_SMD:C_0603_1608Metric, F.Cu at (169.1, 161.0)
- added C110: C_Polarized_Small, Capacitor_THT:CP_Radial_D8.0mm_P3.50mm, F.Cu at (175.6, 156.6)
- added C111: C_Polarized_Small, Capacitor_THT:CP_Radial_D8.0mm_P3.50mm, F.Cu at (175.7, 165.8)
- added C112: 6.8n, Capacitor_SMD:C_0603_1608Metric, F.Cu at (149.1, 179.7)
- added C113: 1n, Capacitor_SMD:C_0603_1608Metric, F.Cu at (151.3, 175.9)
- added C114: 1n, Capacitor_SMD:C_0603_1608Metric, F.Cu at (151.3, 183.4)
- added C115: 100nF, Capacitor_SMD:C_0603_1608Metric, F.Cu at (159.0, 179.8)
- added C116: 39n, Capacitor_SMD:C_0603_1608Metric, F.Cu at (160.4, 179.8)
- added C117: 100nF, Capacitor_SMD:C_0603_1608Metric, F.Cu at (169.1, 179.7)
- added C118: C_Polarized_Small, Capacitor_THT:CP_Radial_D8.0mm_P3.50mm, F.Cu at (175.6, 175.3)
- added C119: C_Polarized_Small, Capacitor_THT:CP_Radial_D8.0mm_P3.50mm, F.Cu at (175.7, 184.5)
- added C87: C_Polarized_Small, Capacitor_THT:CP_Radial_D8.0mm_P3.50mm, F.Cu at (175.7, 119.9)
- added C88: C_Polarized_Small, Capacitor_THT:CP_Radial_D8.0mm_P3.50mm, F.Cu at (175.7, 129.1)
- added C89: 6.8n, Capacitor_SMD:C_0603_1608Metric, F.Cu at (149.1, 124.3)
- added C90: 1n, Capacitor_SMD:C_0603_1608Metric, F.Cu at (151.3, 120.5)
- added C91: 1n, Capacitor_SMD:C_0603_1608Metric, F.Cu at (151.3, 128.0)
- added C92: 100nF, Capacitor_SMD:C_0603_1608Metric, F.Cu at (159.0, 124.4)
- added C93: 39n, Capacitor_SMD:C_0603_1608Metric, F.Cu at (160.5, 124.4)
- added C94: 4.7uF, Capacitor_SMD:C_0603_1608Metric, F.Cu at (110.3, 112.1)
- added C95: 100nF, Capacitor_SMD:C_0603_1608Metric, F.Cu at (169.1, 124.3)
- added C96: 6.8n, Capacitor_SMD:C_0603_1608Metric, F.Cu at (149.1, 142.5)
- added C97: 1n, Capacitor_SMD:C_0603_1608Metric, F.Cu at (151.3, 138.7)
- added C98: 1n, Capacitor_SMD:C_0603_1608Metric, F.Cu at (151.3, 146.2)
- added C99: 100nF, Capacitor_SMD:C_0603_1608Metric, F.Cu at (159.0, 142.6)
- added J24: ACJS-MV35-3, pcm3168a_euro1:Amphenol_ACJS, F.Cu at (190.4, 124.4)
- added J25: ACJS-MV35-3, pcm3168a_euro1:Amphenol_ACJS, F.Cu at (190.3, 142.5)
- added J26: ACJS-MV35-3, pcm3168a_euro1:Amphenol_ACJS, F.Cu at (190.3, 161.0)
- added J27: ACJS-MV35-3, pcm3168a_euro1:Amphenol_ACJS, F.Cu at (190.3, 179.7)
- added R100: 1.1k, Resistor_SMD:R_0603_1608Metric, F.Cu at (151.3, 144.7)
- added R101: 560, Resistor_SMD:R_0603_1608Metric, F.Cu at (151.3, 141.7)
- added R102: 560, Resistor_SMD:R_0603_1608Metric, F.Cu at (151.3, 143.2)
- added R103: 47, Resistor_SMD:R_0603_1608Metric, F.Cu at (159.7, 140.3)
- added R104: 47, Resistor_SMD:R_0603_1608Metric, F.Cu at (159.7, 144.8)
- added R105: 1.1k, Resistor_SMD:R_0603_1608Metric, F.Cu at (162.1, 141.0)
- added R106: 1.1k, Resistor_SMD:R_0603_1608Metric, F.Cu at (162.1, 144.2)
- added R107: 1.1k, Resistor_SMD:R_0603_1608Metric, F.Cu at (169.9, 140.2)
- added R108: 1.1k, Resistor_SMD:R_0603_1608Metric, F.Cu at (169.9, 144.8)
- added R109: 120, Resistor_SMD:R_0603_1608Metric, F.Cu at (171.7, 141.7)
- added R110: 120, Resistor_SMD:R_0603_1608Metric, F.Cu at (171.7, 143.2)
- added R111: 1.1k, Resistor_SMD:R_0603_1608Metric, F.Cu at (146.8, 160.2)
- added R112: 1.1k, Resistor_SMD:R_0603_1608Metric, F.Cu at (146.8, 161.7)
- added R113: 1.1k, Resistor_SMD:R_0603_1608Metric, F.Cu at (151.3, 158.7)
- added R114: 1.1k, Resistor_SMD:R_0603_1608Metric, F.Cu at (151.3, 163.2)
- added R115: 560, Resistor_SMD:R_0603_1608Metric, F.Cu at (151.3, 160.2)
- added R116: 560, Resistor_SMD:R_0603_1608Metric, F.Cu at (151.3, 161.7)
- added R117: 47, Resistor_SMD:R_0603_1608Metric, F.Cu at (159.7, 158.8)
- added R118: 47, Resistor_SMD:R_0603_1608Metric, F.Cu at (159.7, 163.3)
- added R119: 1.1k, Resistor_SMD:R_0603_1608Metric, F.Cu at (162.1, 159.4)
- added R120: 1.1k, Resistor_SMD:R_0603_1608Metric, F.Cu at (162.1, 162.7)
- added R121: 1.1k, Resistor_SMD:R_0603_1608Metric, F.Cu at (169.9, 158.6)
- added R122: 1.1k, Resistor_SMD:R_0603_1608Metric, F.Cu at (169.9, 163.3)
- added R123: 120, Resistor_SMD:R_0603_1608Metric, F.Cu at (171.7, 160.2)
- added R124: 120, Resistor_SMD:R_0603_1608Metric, F.Cu at (171.7, 161.7)
- added R125: 1.1k, Resistor_SMD:R_0603_1608Metric, F.Cu at (146.8, 178.9)
- added R126: 1.1k, Resistor_SMD:R_0603_1608Metric, F.Cu at (146.8, 180.4)
- added R127: 1.1k, Resistor_SMD:R_0603_1608Metric, F.Cu at (151.3, 177.4)
- added R128: 1.1k, Resistor_SMD:R_0603_1608Metric, F.Cu at (151.3, 181.9)
- added R129: 560, Resistor_SMD:R_0603_1608Metric, F.Cu at (151.3, 178.9)
- added R130: 560, Resistor_SMD:R_0603_1608Metric, F.Cu at (151.3, 180.4)
- added R131: 47, Resistor_SMD:R_0603_1608Metric, F.Cu at (159.7, 177.5)
- added R132: 47, Resistor_SMD:R_0603_1608Metric, F.Cu at (159.7, 182.0)
- added R133: 1.1k, Resistor_SMD:R_0603_1608Metric, F.Cu at (162.1, 178.2)
- added R134: 1.1k, Resistor_SMD:R_0603_1608Metric, F.Cu at (162.1, 181.4)
- added R135: 1.1k, Resistor_SMD:R_0603_1608Metric, F.Cu at (169.9, 177.4)
- added R136: 1.1k, Resistor_SMD:R_0603_1608Metric, F.Cu at (169.9, 182.0)
- added R137: 120, Resistor_SMD:R_0603_1608Metric, F.Cu at (171.7, 178.9)
- added R138: 120, Resistor_SMD:R_0603_1608Metric, F.Cu at (171.7, 180.4)
- added R82: 1.1k, Resistor_SMD:R_0603_1608Metric, F.Cu at (146.8, 123.5)
- added R83: 1.1k, Resistor_SMD:R_0603_1608Metric, F.Cu at (146.8, 125.0)
- added R84: 1.1k, Resistor_SMD:R_0603_1608Metric, F.Cu at (151.3, 122.0)
- added R85: 1.1k, Resistor_SMD:R_0603_1608Metric, F.Cu at (151.3, 126.5)
- added R86: 560, Resistor_SMD:R_0603_1608Metric, F.Cu at (151.3, 123.5)
- added R87: 560, Resistor_SMD:R_0603_1608Metric, F.Cu at (151.3, 125.0)
- added R88: 47, Resistor_SMD:R_0603_1608Metric, F.Cu at (159.7, 122.2)
- added R89: 47, Resistor_SMD:R_0603_1608Metric, F.Cu at (159.7, 126.7)
- added R90: 22, Resistor_SMD:R_0603_1608Metric, F.Cu at (124.4, 162.8)
- added R91: 1.1k, Resistor_SMD:R_0603_1608Metric, F.Cu at (169.9, 122.0)
- added R92: 1.1k, Resistor_SMD:R_0603_1608Metric, F.Cu at (169.9, 126.7)
- added R93: 1.1k, Resistor_SMD:R_0603_1608Metric, F.Cu at (162.1, 122.8)
- added R94: 1.1k, Resistor_SMD:R_0603_1608Metric, F.Cu at (162.1, 126.0)
- added R95: 120, Resistor_SMD:R_0603_1608Metric, F.Cu at (171.7, 123.6)
- added R96: 120, Resistor_SMD:R_0603_1608Metric, F.Cu at (171.7, 125.1)
- added R97: 1.1k, Resistor_SMD:R_0603_1608Metric, F.Cu at (146.8, 141.7)
- added R98: 1.1k, Resistor_SMD:R_0603_1608Metric, F.Cu at (146.8, 143.2)
- added R99: 1.1k, Resistor_SMD:R_0603_1608Metric, F.Cu at (151.3, 140.2)
- added U16: OPA1637, Package_SO:SOIC-8_3.9x4.9mm_P1.27mm, F.Cu at (155.5, 124.4)
- added U17: OPA1637, Package_SO:SOIC-8_3.9x4.9mm_P1.27mm, F.Cu at (165.6, 124.4)
- added U18: OPA1637, Package_SO:SOIC-8_3.9x4.9mm_P1.27mm, F.Cu at (155.5, 142.6)
- added U19: OPA1637, Package_SO:SOIC-8_3.9x4.9mm_P1.27mm, F.Cu at (165.6, 142.5)
- added U20: OPA1637, Package_SO:SOIC-8_3.9x4.9mm_P1.27mm, F.Cu at (155.5, 161.0)
- added U21: OPA1637, Package_SO:SOIC-8_3.9x4.9mm_P1.27mm, F.Cu at (165.6, 161.0)
- added U22: OPA1637, Package_SO:SOIC-8_3.9x4.9mm_P1.27mm, F.Cu at (155.5, 179.8)
- added U23: OPA1637, Package_SO:SOIC-8_3.9x4.9mm_P1.27mm, F.Cu at (165.6, 179.7)
- C31: value C_Small -> C_Polarized_Small; footprint Capacitor_SMD:C_0603_1608Metric -> Capacitor_THT:CP_Radial_D8.0mm_P3.50mm
- C32: value 100nF -> 1n
- J1: value Conn_02x04_Odd_Even -> ACJS-MV35-3; footprint Connector_PinHeader_2.54mm:PinHeader_2x04_P2.54mm_Vertical -> pcm3168a_euro1:Amphenol_ACJS
- R1: moved to F.Cu
- R11, R13, R14, R16: value 0 -> 220k 5%
- R2: value 220k 5% -> 1.1k; moved to F.Cu
- R34: value 0 -> 22k
- R60: value 1.1k -> 22
- moved R14 200.2 mm to (274.6, 138.3)
- moved R11 198.9 mm to (274.6, 133.3)
- moved R13 192.1 mm to (274.6, 135.8), turned to 0 degrees
- moved R16 184.8 mm to (274.6, 140.8)
- moved J10 175.6 mm to (140.9, 200.3), turned to 90 degrees
- moved R27 169.3 mm to (140.1, 194.5)
- moved C20 165.4 mm to (143.1, 193.7), turned to 0 degrees
- moved U3 164.6 mm to (141.0, 190.9), turned to -90 degrees
- moved C19 161.4 mm to (138.7, 188.0), turned to 180 degrees
- moved R26 160.0 mm to (143.3, 188.0)
- moved R25 160.0 mm to (141.0, 187.2), turned to -90 degrees
- moved J12 144.8 mm to (116.5, 200.3), turned to 90 degrees
- moved R33 138.9 mm to (115.7, 194.5)
- moved C24 134.7 mm to (118.7, 193.7), turned to 0 degrees
- moved U5 134.3 mm to (116.6, 190.9), turned to -90 degrees
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Connections:
- C31 pad 2: GND -> Net-(J1-Pin_4)
- C32 pad 1: VDD -> Net-(C32-Pad1)
- C32 pad 2: GND -> Net-(C32-Pad2)
- C67 pad 2: Net-(J20-Pin_3) -> Net-(J1-Pin_3)
- J1 pad 1: /MODE -> GND
- J1 pad 2: GND -> unconnected-(J1-Pin_2-Pad2)
- J1 pad 3: /MODE -> Net-(J1-Pin_3)
- J1 pad 5: /MODE -> unconnected-(J1-Pin_5-Pad5)
- J13 pad 1: Net-(D3-K) -> Net-(J13-In)
- J15 pad 1: Net-(D4-K) -> Net-(J15-In)
- R1 pad 1: GND -> Net-(U1-MODE)
- R1 pad 2: Net-(J1-Pin_4) -> GND
- R11 pad 1: /lrclk_slave/OUT -> Net-(U1-MDO_ADR1_MD1)
- R11 pad 2: /LRCK -> GND
- R13 pad 1: /bck_master/IN -> VDD
- R13 pad 2: /BCK -> Net-(U1-MS_ADR0_MD0)
- R14 pad 1: /lrck_master/IN -> Net-(U1-MDI_SDA_DEMP)
- R14 pad 2: /LRCK -> GND
- R16 pad 1: /mclk/OUT1 -> VDD
- R16 pad 2: /SCKI -> Net-(U1-MC_SCL_FMT)
- R2 pad 1: GND -> Net-(C68-Pad1)
- R2 pad 2: Net-(J2-Pin_4) -> Net-(C32-Pad1)
- R30 pad 2: /lrclk_slave/OUT -> /clk_in/OUT
- R35 pad 1: Net-(D3-K) -> Net-(R35-Pad1)
- R37 pad 2: /mclk/OUT1 -> Net-(J13-In)
- R38 pad 1: Net-(R38-Pad1) -> Net-(Y1-OUT)
- R38 pad 2: /mclk/OUT2 -> Net-(R35-Pad1)
- R42 pad 1: Net-(D4-K) -> /clk_in/OUT
- R42 pad 2: Net-(C31-Pad1) -> Net-(C33-Pad1)
- R43 pad 2: Net-(C31-Pad1) -> Net-(C33-Pad1)
- R44 pad 2: /external_clock/OUT -> Net-(J15-In)
- R58 pad 2: Net-(C66-Pad1) -> Net-(C31-Pad1)
- R60 pad 1: Net-(C68-Pad1) -> /bck_master/IN
- R60 pad 2: Net-(C69-Pad1) -> Net-(U1-BCKAD)
- R62 pad 1: Net-(C69-Pad2) -> Net-(C32-Pad2)
- R64 pad 2: Net-(C69-Pad1) -> Net-(C32-Pad1)
- U1 pad 25: unconnected-(U1-VOUT4+-Pad25) -> /VOUT4+
- U1 pad 26: unconnected-(U1-VOUT4--Pad26) -> /VOUT4-
- U1 pad 27: unconnected-(U1-VOUT3+-Pad27) -> /VOUT3+
- U1 pad 28: unconnected-(U1-VOUT3--Pad28) -> /VOUT3-
- U1 pad 29: unconnected-(U1-VOUT2+-Pad29) -> /VOUT2+
- U1 pad 30: unconnected-(U1-VOUT2--Pad30) -> /VOUT2-
- U1 pad 31: unconnected-(U1-VOUT1+-Pad31) -> /VOUT1+
- U1 pad 32: unconnected-(U1-VOUT1--Pad32) -> /VOUT1-
- U1 pad 35: /LRCK -> /lrck_master/IN
- U1 pad 36: /BCK -> /bck_master/IN
- U1 pad 41: /SCKI -> /clk_in/OUT
- U1 pad 42: /FMT_SCL -> Net-(U1-MC_SCL_FMT)
- U1 pad 43: /DEMP_SDA -> Net-(U1-MDI_SDA_DEMP)
- U1 pad 44: /MD1 -> Net-(U1-MDO_ADR1_MD1)
- U1 pad 45: /MD0 -> Net-(U1-MS_ADR0_MD0)
- U1 pad 48: /MODE -> Net-(U1-MODE)
- U1 pad 6: /LRCK -> Net-(U1-LRCKAD)
- U1 pad 7: /BCK -> Net-(U1-BCKAD)
- U13 pad 5: Net-(C69-Pad1) -> Net-(C32-Pad1)
- U13 pad 8: Net-(C69-Pad2) -> Net-(C32-Pad2)
- U9 pad 2: Net-(C31-Pad1) -> Net-(C33-Pad1)
- Y1 pad 3: /oscillator/OSC_OUT -> Net-(Y1-OUT)
Routing:
- net /dout1/IN: track 83.7 -> 2.04 mm, vias 2 -> 0
- net VCOMAD: track 100.6 -> 26.8 mm, vias 7 -> 0
- net /LRCK: track 67.9 -> 0.00 mm, vias 2 -> 0
- net /BCK: track 58.8 -> 0.00 mm, vias 2 -> 0
- net /SCKI: track 56.3 -> 0.00 mm
- net /mclk/OUT1: track 49.0 -> 0.00 mm
- net /din1/OUT: track 49.1 -> 2.04 mm
- net Net-(J1-Pin_4): track 0.00 -> 29.7 mm
- net Net-(J1-Pin_3): track 0.00 -> 29.5 mm
- net Net-(J20-Pin_4): track 25.4 -> 0.00 mm
- net Net-(J20-Pin_3): track 24.7 -> 0.00 mm
- net Net-(J25-Pin_3): track 0.00 -> 16.8 mm
- net Net-(J24-Pin_3): track 0.00 -> 16.8 mm
- net Net-(J26-Pin_3): track 0.00 -> 16.8 mm
- net Net-(J27-Pin_3): track 0.00 -> 16.8 mm
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Other:
- board size 196 x 128.4 mm -> 141.8 x 132.5 mm
- board text removed: "BCK MST"
- board text removed: "BCK SLV"
- board text removed: "DEMP"
- board text removed: "DIN"
- board text removed: "DOUT"
- board text removed: "EXT CLK"
- board text removed: "FMT"
- board text removed: "IN"
- board text removed: "LRCK MST"
- board text removed: "LRCLK SLV"
- board text removed: "MD0"
- board text removed: "MD1"
- board text removed: "MODE"
- board text removed: "OSC"
- board text removed: "OUT"
- board text removed: "SCKI SLV"
- board text removed: "SCL"
- board text removed: "SDA"

Commit message: WIP layout
Parts:
- J18: footprint Connector_PinHeader_2.54mm:PinHeader_2x08_P2.54mm_Vertical -> Connector_PinSocket_2.54mm:PinSocket_2x08_P2.54mm_Vertical; moved to B.Cu
- R1, R11, R13, R14, R16, R21: moved to B.Cu
- moved J18 217.6 mm to (58.2, 115.2)
- moved C49 214.8 mm to (65.7, 104.7), turned to -90 degrees
- moved C47 212.7 mm to (67.4, 104.7), turned to -90 degrees
- moved C42 208.0 mm to (66.2, 109.1), turned to -90 degrees
- moved L1 206.0 mm to (64.8, 102.5)
- moved C43 205.7 mm to (62.6, 104.8)
- moved R56 204.3 mm to (61.8, 102.5)
- moved C45 198.9 mm to (74.9, 109.1), turned to -90 degrees
- moved C44 197.4 mm to (71.7, 102.1), turned to -90 degrees
- moved R57 192.6 mm to (72.7, 99.8), turned to 0 degrees
- moved C59 191.1 mm to (96.0, 116.0)
- moved U12 190.9 mm to (90.7, 109.1), turned to 180 degrees
- moved C65 188.5 mm to (95.9, 111.3), turned to -90 degrees
- moved C62 184.6 mm to (97.5, 111.3), turned to -90 degrees
- moved C46 182.5 mm to (90.0, 102.0), turned to 90 degrees
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Connections:
- C1 pad 1: +3.3V -> VDD
- C2 pad 1: +3.3V -> VDD
- C3 pad 2: +3.3V -> VDD
- C4 pad 2: +3.3V -> VDD
- C59 pad 1: +3.3V -> VDD
- C62 pad 1: +3.3V -> VDD
- C65 pad 1: +3.3V -> VDD
- U1 pad 12: +3.3V -> VDD
- U1 pad 46: +3.3V -> VDD
- U12 pad 2: +3.3V -> VDD
Routing:
- net /VOUT4+: track 0.00 -> 42.8 mm
- net /VOUT1+: track 0.00 -> 40.8 mm
- net Net-(U1-VCOMDA): track 4.39 -> 45.0 mm, vias 0 -> 1
- net /VOUT4-: track 0.00 -> 39.2 mm
- net /VOUT1-: track 0.00 -> 36.5 mm
- net /VOUT3+: track 0.00 -> 25.6 mm
- net /VOUT2+: track 0.00 -> 23.1 mm
- net /VOUT3-: track 0.00 -> 21.7 mm
- net /VOUT2-: track 0.00 -> 20.3 mm
- net +3.3V: track 9.95 -> 0.00 mm, vias 3 -> 0
- net VDD: track 8.64 -> 18.6 mm, vias 6 -> 9
- net Net-(R24-Pad1): track 2.45 -> 0.00 mm
- net /dout1/IN: track 2.04 -> 0.00 mm
- net /lrck_master/IN: track 1.30 -> 0.00 mm
- added copper zone on In2.Cu, net +5V
- added copper zone on In2.Cu, net VDD
Other:
- board size 141.8 x 132.5 mm -> 153.7 x 132.5 mm
- copper layers 2 -> 4

Commit message: WIP layout
Parts:
- added H1: MountingHole_Pad, MountingHole:MountingHole_3.2mm_M3_DIN965_Pad, F.Cu at (91.3, 71.7)
- added H2: MountingHole_Pad, MountingHole:MountingHole_3.2mm_M3_DIN965_Pad, F.Cu at (91.3, 194.2)
- added H3: MountingHole_Pad, MountingHole:MountingHole_3.2mm_M3_DIN965_Pad, F.Cu at (167.5, 71.7)
- added H4: MountingHole_Pad, MountingHole:MountingHole_3.2mm_M3_DIN965_Pad, F.Cu at (243.7, 71.7)
- added H5: MountingHole_Pad, MountingHole:MountingHole_3.2mm_M3_DIN965_Pad, F.Cu at (167.5, 194.2)
- added H6: MountingHole_Pad, MountingHole:MountingHole_3.2mm_M3_DIN965_Pad, F.Cu at (243.7, 194.2)
- added J16: Conn_01x02_Pin, Connector_PinHeader_2.54mm:PinHeader_1x02_P2.54mm_Vertical, F.Cu at (155.4, 94.7)
- added R3: 0, Resistor_SMD:R_0603_1608Metric, F.Cu at (96.8, 71.7)
- added R4: 0, Resistor_SMD:R_0603_1608Metric, F.Cu at (96.8, 194.2)
- added R5: 0, Resistor_SMD:R_0603_1608Metric, F.Cu at (173.4, 71.6)
- added R6: 0, Resistor_SMD:R_0603_1608Metric, F.Cu at (238.1, 71.7)
- added R7: 0, Resistor_SMD:R_0603_1608Metric, F.Cu at (161.3, 194.2)
- added R8: 0, Resistor_SMD:R_0603_1608Metric, F.Cu at (237.4, 194.2)
- moved C59 48.8 mm to (128.7, 79.8), turned to 90 degrees
- moved U12 48.7 mm to (134.0, 86.6), turned to 0 degrees
- moved C46 45.5 mm to (134.7, 93.8), turned to -90 degrees
- moved C105 44.6 mm to (191.2, 139.5)
- moved C106 44.6 mm to (191.2, 147.0)
- moved C110 44.6 mm to (215.6, 138.8)
- moved C117 44.6 mm to (209.1, 162.0)
- moved C38 44.6 mm to (139.1, 123.9)
- moved C73 44.6 mm to (130.0, 141.2)
- moved C81 44.6 mm to (129.7, 167.8)
- moved C98 44.6 mm to (191.2, 128.5)
- moved J10 44.6 mm to (179.1, 182.7)
- moved J27 44.6 mm to (230.3, 162.0)
- moved J8 44.6 mm to (160.0, 152.7)
- moved R1 44.6 mm to (158.0, 125.6)
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Connections:
- C13 pad 1: Net-(U1-VCOMDA) -> VCOMDA
- U1 pad 15: Net-(U1-VCOMDA) -> VCOMDA
Routing:
- net VCOMDA: track 0.00 -> 172.2 mm, vias 0 -> 22
- net VCOMAD: track 26.8 -> 98.1 mm, vias 0 -> 11
- net Net-(C42-Pad1): track 0.00 -> 59.0 mm
- net Net-(U1-VCOMDA): track 45.0 -> 0.00 mm, vias 1 -> 0
- net Net-(R24-Pad1): track 0.00 -> 41.9 mm
- net /clk_in/OUT: track 7.83 -> 45.2 mm
- net /dout1/IN: track 0.00 -> 33.9 mm
- net /lrck_master/IN: track 0.00 -> 30.6 mm
- net /bck_master/IN: track 0.09 -> 21.2 mm
- net +5V: track 26.0 -> 41.4 mm, vias 5 -> 17
- net Net-(U12-VI): track 0.00 -> 12.8 mm
- net VDD: track 18.6 -> 29.3 mm
- net Net-(J16-Pin_1): track 0.00 -> 7.65 mm
- net Net-(D1-K): track 0.00 -> 7.53 mm
- net Net-(C17-Pad1): track 0.00 -> 5.87 mm
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- added copper zone on F.Cu, net +5V
- added copper zone on F.Cu, net GND
- added copper zone on In1.Cu, net GND
Other:
- board size 153.7 x 132.5 mm -> 162.7 x 132.5 mm
- board text added: "+5V"
- board text added: "BCK OUT"
- board text added: "CLK IN"
- board text added: "CLK OUT"
- board text added: "DIN"
- board text added: "DOUT"
- board text added: "LRCK OUT"
- board text added: "NATURAL SYSTEMS TDM44 REV A"
- board text added: "OSC OUT"
- board text added: "RST"
- board text added: "SYNC"

Commit message: WIP layout
Parts:
- removed R21: 220k 5%, Resistor_SMD:R_0603_1608Metric
- moved R19 15.6 mm to (172.2, 154.8)
- moved J8 10.7 mm to (169.6, 157.6)
- moved R13 6.07 mm to (159.1, 120.2)
- moved R11 5.59 mm to (160.7, 120.2)
- moved R1 5.55 mm to (157.5, 120.1)
- moved R16 3.68 mm to (163.8, 120.1)
- moved R14 3.62 mm to (162.2, 120.2)
- moved C34 2.72 mm to (159.4, 91.8)
- moved C15 0.88 mm to (156.0, 142.0)
- moved C16 0.88 mm to (156.0, 139.6)
Connections:
- C10 pad 2: Net-(U1-VCCAD1) -> +5V
- C11 pad 1: Net-(U1-VCCAD1) -> +5V
- C12 pad 1: Net-(U1-VCCAD1) -> +5V
- C5 pad 2: Net-(U1-VCCDA2) -> +5V
- C6 pad 2: Net-(U1-VCCDA1) -> +5V
- C7 pad 1: Net-(U1-VCCDA1) -> +5V
- C8 pad 1: Net-(U1-VCCDA2) -> +5V
- C9 pad 2: Net-(U1-VCCAD1) -> +5V
- U1 pad 13: Net-(U1-ZERO) -> unconnected-(U1-ZERO-Pad13)
- U1 pad 14: Net-(U1-VCCDA1) -> +5V
- U1 pad 3: Net-(U1-VCCAD1) -> +5V
- U1 pad 34: Net-(U1-VCCDA2) -> +5V
- U1 pad 49: Net-(U1-VCCAD1) -> +5V
Routing:
- net VDD: track 29.3 -> 184.7 mm, vias 9 -> 18
- net +5V: track 41.4 -> 108.8 mm, vias 17 -> 34
- net GND: track 21.6 -> 73.9 mm, vias 51 -> 125
- net Net-(J8-Pin_2): track 0.00 -> 23.5 mm, vias 0 -> 1
- net /lrck_master/IN: track 30.6 -> 50.2 mm, vias 0 -> 2
- net /bck_master/IN: track 21.2 -> 40.8 mm, vias 0 -> 2
- net Net-(U1-MS_ADR0_MD0): track 0.00 -> 12.0 mm, vias 0 -> 1
- net Net-(U1-MODE): track 0.00 -> 11.7 mm, vias 0 -> 1
- net Net-(U1-MDO_ADR1_MD1): track 0.00 -> 11.3 mm, vias 0 -> 1
- net Net-(U1-MDI_SDA_DEMP): track 0.00 -> 10.7 mm, vias 0 -> 1
- net Net-(U1-MC_SCL_FMT): track 0.00 -> 10.3 mm, vias 0 -> 1
- net Net-(U1-VREFAD2): track 0.00 -> 6.49 mm
- net Net-(U1-VCCDA1): track 6.36 -> 0.00 mm
- net VCOMAD: track 98.1 -> 104.0 mm
- net Net-(U1-VCCDA2): track 5.48 -> 0.00 mm
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- added copper zone on B.Cu, net GND
