File: out_amp.kicad_sch (KiCad schematic)
At the start: 17 parts, among them J17 ACJS-MV35-3, U11 OPA1637

Commit message: redoing file add
Parts:
- removed J17: ACJS-MV35-3, pcm3168a_euro1:Amphenol_ACJS, symbol Connector:Conn_01x05_Socket
- added J24: ACJS-MV35-3, pcm3168a_euro1:Amphenol_ACJS, symbol Connector:Conn_01x05_Socket
- renumbered C35 to C87, C36 to C88, C37 to C89, C38 to C90, C39 to C91, C40 to C92, C41 to C93, R48 to R82, R49 to R83, R50 to R84, R51 to R85, R52 to R86, R53 to R87, R54 to R88, R55 to R89, U11 to U16
Connections:
- net OUT+ is gone; now on an unnamed net: C93.2, R89.2
- net OUT- is gone; now on an unnamed net: C93.1, R88.1
- net GND: now also J24.1 (Pin_1)
- net at C87.1: no longer R82.2
- net at C87.2: now also J24.3 (Pin_3)
- net at C88.2: now also J24.4 (Pin_4)
- net at C88.1: no longer R83.1
- net VCOMAD renamed VCOMDA
- new net IN+: R82.2
- new net IN-: R83.1
Other:
- note removed: "connectors: amphenol ACJS-MV35-3 same sky SJ3-35053A"
- note removed: "wire up based on chosen connector"
- moved on the sheet: C87, C88

Commit message: WIP layout
Parts:
- added C101: 100nF, Capacitor_SMD:C_0603_1608Metric, symbol Device:C_Small
- added R105, R106, R107, R108: 1.1k, Resistor_SMD:R_0603_1608Metric, symbol Device:R_Small
- added R109, R110: 120, Resistor_SMD:R_0603_1608Metric, symbol Device:R_Small
- added U19: OPA1637, Package_SO:SOIC-8_3.9x4.9mm_P1.27mm, symbol Amplifier_Operational:LMH6551MA
- renumbered C93 to C100, C87 to C102, C88 to C103, C89 to C96, C90 to C97, C91 to C98, C92 to C99, J24 to J25, R85 to R100, R86 to R101, R87 to R102, R88 to R103, R89 to R104, R82 to R97, R83 to R98, R84 to R99, U16 to U18
Connections:
- net +5V: now also C101.1, U19.3 (V+)
- net GND: now also C101.2, U19.6 (V-)
- net VCOMDA: now also U19.2 (VCM)
- net at C100.1, R103.1: now also R105.2; no longer C102.1
- net at C102.2: now also J25.4 (Pin_4); no longer J25.3 (Pin_3)
- net at C100.2, R104.2: now also R106.2; no longer C103.1
- net at C103.2: now also J25.3 (Pin_3); no longer J25.4 (Pin_4)
- new net: R105.1, R107.1, U19.8 (+)
- new net: C102.1, R109.1
- new net: C103.1, R110.1
- new net: R108.1, R110.2, U19.4 (+)
- new net: R106.1, R108.2, U19.1 (-)
- new net: R107.2, R109.2, U19.5 (-)
Other:
- note added: "120 out resistors current limit < 50 mA in case outputs are shorted to ground"
- note added: "consider series resistance on output. need to understand case where the output is connected to an unbalanced input. Not sure if this connects one of the signals (ring, minus) to ground or leaves it open see: https://www.ranecommercial.com/legacy/note110.html "sound system interconnection""
- note added: "pin 3 should be + pin 4 should be - pin 1 is shield (gnd) flipping the connections at the input compensates for the amp inversion"
- note removed: "- use nichicon caps for signal path, "nichicon MUSE" covers a lot of high quality audio grade caps - bipolar caps make the most sense for AC coupling - alternatively, polar caps, + side facing the diffamp, and then have a pull down to ground on the minus side - the pulldown will help if the incoming signal has outputs that are AC couples, so the common mode level would forced to ground by the pul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"
- moved on the sheet: C100, C102, C103, C96, C97, C98, C99, J25, R100, R101, R102, R103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
