File: out_amp.kicad_sch (KiCad schematic)
At the start: 25 parts, among them J25 ACJS-MV35-3, U18 OPA1637, U19 OPA1637

Commit message: DONE. now exporting gerbers
Parts:
- C100: footprint Capacitor_SMD:C_0603_1608Metric -> Capacitor_SMD:C_0805_2012Metric
- U18, U19: footprint Package_SO:SOIC-8_3.9x4.9mm_P1.27mm -> Package_SO:MSOP-8_3x3mm_P0.65mm
Changed lines of the file:
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@@
 			"QIF/1G5iAACQ+WrUbmIAABCqlNRuYgAAAN5b1G5iAABAEZbUbmIAACAKWtRuYgAA4H+C1G5iAABQ"
 			"OFTUbmIAAACgYdRuYgAAwEEl1W5iAAAwXGbUbmIAAKBRwNRuYgAAEO0g1W5iAAAg7ZfUbmIAAJCo"
-			"mdRuYgAAULwg1W5iAAAAulbUbmIAAAA9w9RuYgAAgDFc1G5iAA=="
+			"mdRuYgAAULwg1W5iAAAAulbUbmIAAAA9w9RuYgAAgDFc1G5iAAAAAAAAAAAAAAAAAAAAAAAAAAAA"
+			"AAAAAAAAAAAAAAAAAAAAAAAAAAAAAAAAAAAAAAAAAAAAAAAAAAAAAAAAAAAAAAAAAAAAAAAAAAAA"
+			"AAAAAAAAAAAAAAAAAAAAAAAAAAAAAAAAAAAAAAAAAAAAAAAAAAAAAAAAAAAAAAAAAAAAAAAAAAAA"
+			"AAAAAAAAAAAAAAAAAAAAAAAAAAAAAAAAAAAAAAAAAAAAAAAAAAAAAAAAAAAAAAAAAAAAAAAAAAAA"
+			"AAAAAAAAAAAAAAAAAAAAAAAAAAAAAAAAAAAAAAAAAAAAAAAAAAAAAAAAAAAAAAAAAAAAAAAAAAAA"
+			"AAAAAAAAAAAAAAAAAAAAAAAAAAAAAAAAAAAAAAAAAAAAAAAAAAAAAAAAAAAAAAAAAAAAAAAAAAAA"
+			"AAAAAAAAAAAAAAAAAAAAAAAAAAAAAAAAAAAAAAAAAAAAAAAAAAAAAAAAAAAAAAAAAAAAAAAAAAAA"
+			"AAAAAAAAAAAAAAAAAAAAAAAAAAAAAAAAAAAAAAAAAAAAAAAAAAAAAAAAAAAAAAAAAAAAAAAAAAAA"
+			"AAAAAAAAAAAAAAAAAAAAAAAAAAAAAAAAAAAAAAAAAAAAAAAAAAAAAAAAAAAAAAAAAAAAAAAAAAAA"
+			"AAAAAAAAAAAAAAAAAAAAAAAAAAAAAAAAAAAAAAAAAAAAAAAAAAAAAAAAAAAAAAAAAAAAAAAAAAAA"
+			"AAAAAAAAAAAAAAAAAAAAAAAAAAAAAAAAAAAAAAAAAAAAAAAAAAAAAAAAAAAAAAAAAAAAAAAAAAAA"
+			"AAAAAAAAAAAAAAAAAAAAAAAAAAAAAAAAAAAAAAAAAAAAAAAAAAAAAAAAAAAAAAAAAAAAAAAAAAAA"
+			"AAAAAAAAAAAAAAAAAAAAAAAAAAAAAAAAAAAAAAAAAAAAAAAAAAAAAAAAAAAAAAAAAAAAAAAAAAAA"
+			"AAAAAAAAAAAAAAAAAAAAAAAAAAAAAAAAAAAAAAAAAAAAAAAAAAAAAAAAAAAAAAAAAAAAAAAAAAAA"
+			"AAAAAAAAAAAAAAAAAAAAAAAAAAAAAAAAAAAAAAAAAAAAAAAAAAAAAAAAAAAAAAAAAAAAAAAAAAAA"
+			"AAAAAAAAAAAAAAAAAAAAAAAAAAAAAAAAAAAAAAAAAAAAAAAAAAAAAAAAAAAAAAAAAAAAAAAAAAAA"
+			"AAAAAAAAAAAAAAAAAAAAAAAAAAAAAAAAAAAAAAAAAAAAAAAAAAAAAAAAAAAAAAAAAAAAAAAAAAAA"
+			"AAAAAAAAAAAAAAAAAAAAAAAAAAAAAAAAAAAAAAAAAAAAAAAAAAAAAAAAAAAAAAAAAAAAAAAAAAAA"
+			"AAAAAAAAAAAAAAAAAAAAAAAAAAAAAAAAAAAAAAAAAAAAAAAAAAAAAAAAAAAdAAAAAAAAAH4AAAAA"
+			"AAAAEBOHn6hXAAAeAAAAAAAAAB4AAAAAAAAAeCu2dqhXAAAwlGWIqFcAABkAAAAAAAAAGQAAAAAA"
+			"AAAAAAAAAAAAAPChynmoVwAAGgAAAAAAAAAaAAAAAAAAALgrtnaoVwAAcG0cdahXAAAcAAAAAAAA"
+			"ABwAAAAAAAAAAAAAAAAAAAAw1ptqqFcAABgAAAAAAAAAGAAAAAAAAAAAAAAAAAAAAACjV4eoVwAA"
+			"EAAAAAAAAAAQAAAAAAAAAAEAAAAAAAAAgBimiKhXAAATAAAAAAAAABMAAAAAAAAAAQAAAAAAAADg"
+			"tJ+YqFcAABEAAAAAAAAAEQAAAAAAAAAAAAAAAAAAAMC/R5+oVwAAEQAAAAAAAAARAAAAAAAAAAAA"
+			"AAAAAAAA0PwFdKhXAAAUAAAAAAAAABQAAAAAAAAAAAAAAAAAAABwMo6YqFcAABoAAAAAAAAAGgAA"
+			"AAAAAABAek1rqFcAAHBw53SoVwAAHgAAAAAAAAAeAAAAAAAAAJwxAACcEgAA0FaniKhXAAAkAAAA"
+			"AAAAACQAAAAAAAAAKzMAAAAAAAAwzFWhqFcAACgAAAAAAAAAKAAAAAAAAADQl6x2qFcAAIDqzp+o"
+			"VwAAKQAAAAAAAAApAAAAAAAAACAetnaoVwAA4Lj1dqhXAAAkAAAAAAAAACQAAAAAAAAAAAAAAAAA"
+			"AACAMYpqqFcAACUAAAAAAAAAJQAAAAAAAAAQdwAAAAAAADAvtXaoVwAAJwAAAAAAAAAnAAAAAAAA"
+			"ADAAAAAAAAAAYEvze6hXAAAjAAAAAAAAACMAAAAAAAAA//////////9QON9yqFcAAB4AAAAAAAAA"
+			"HgAAAAAAAABwtYV8qFcAALD5RoioVwAAIwAAAAAAAAAjAAAAAAAAAJAttnaoVwAAwBxRnahXAAAp"
+			"AAAAAAAAACkAAAAAAAAAAAAAAAAAAABgVL+GqFcAAC0AAAAAAAAALQAAAAAAAAAQdwAAAAAAAHA8"
+			"KaCoVwAALgAAAAAAAAAuAAAAAAAAADAAAAAAAAAAcM9rh6hXAAApAAAAAAAAACkAAAAAAAAAaQAA"
+			"AG4AAADQ6iqgqFcAACoAAAAAAAAAKgAAAAAAAAB0AAAAYQAAABBwZXOoVwAALAAAAAAAAAAsAAAA"
+			"AAAAACEAAAAAAAAAQOM7aqhXAAAoAAAAAAAAACgAAAAAAAAAcAAAAAAAAAAAnP93qFcAAB8AAAAA"
+			"AAAAHwAAAAAAAAAAAAAAAAAAAOCSpGqoVwAAGgAAAAAAAAAaAAAAAAAAAAAAAAAAAAAA4KOhdahX"
+			"AAAbAAAAAAAAABsAAAAAAAAAAAAAAAAAAABAOJWgqFcAAB0AAA=="
 		)
 	)
@@
 			)
 		)
-		(property "Footprint" "Package_SO:SOIC-8_3.9x4.9mm_P1.27mm"
+		(property "Footprint" "Package_SO:MSOP-8_3x3mm_P0.65mm"
 			(at 199.39 114.3 0)
 			(effects
@@
 			)
 		)
-		(property "Footprint" "Capacitor_SMD:C_0603_1608Metric"
+		(property "Footprint" "Capacitor_SMD:C_0805_2012Metric"
 			(at 142.24 99.06 0)
 			(effects
@@
 			)
 		)
-		(property "Footprint" "Package_SO:SOIC-8_3.9x4.9mm_P1.27mm"
+		(property "Footprint" "Package_SO:MSOP-8_3x3mm_P0.65mm"
 			(at 104.14 114.3 0)
 			(effects

Commit message: added part numbers
Parts:
- C100: PN (none) -> GRM2195C2A393GE01J
- C101, C99: PN (none) -> GCJ188R71H104KA12D
- C96: PN (none) -> C0603X682F5GECTU
- C97, C98: PN (none) -> GCM1885C2A102FA16D
- R100, R105, R106, R107, R108, R97, R98, R99: PN (none) -> ERA-3AEB112V
- R101, R102: PN (none) -> ERA-3AEB561V
- R103, R104: PN (none) -> ERA-3AEB470V
- R109, R110: PN (none) -> ERA-3AEB121V
- U18, U19: PN (none) -> OPA1637DGKR
Changed lines of the file:
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@@
 			"AAAAACEAAAAAAAAAQOM7aqhXAAAoAAAAAAAAACgAAAAAAAAAcAAAAAAAAAAAnP93qFcAAB8AAAAA"
 			"AAAAHwAAAAAAAAAAAAAAAAAAAOCSpGqoVwAAGgAAAAAAAAAaAAAAAAAAAAAAAAAAAAAA4KOhdahX"
-			"AAAbAAAAAAAAABsAAAAAAAAAAAAAAAAAAABAOJWgqFcAAB0AAA=="
+			"AAAbAAAAAAAAABsAAAAAAAAAAAAAAAAAAABAOJWgqFcAAB0AAAAAAAAAAAAAAAAAAAAAAAAAAAAA"
+			"AAAAAAAAAAAAAAAAAAAAAAAAAAAAAAAAAAAAAAAAAAAAAAAAAAAAAAAAAAAAAAAAAAAAAAAAAAAA"
+			"AAAAAAAAAAAAAAAAAAAAAAAAAAAAAAAAAAAAAAAAAAAAAAAAAAAAAAAAAAAAAAAAAAAAAAAAAAAA"
+			"AAAAAAAAAAAAAAAAAAAAAAAAAAAAAAAAAAAAAAAAAAAAAAAAAAAAAAAAAAAAAAAAAAAAAAAAAAAA"
+			"AAAAAAAAAAAAAAAAAAAAAAAAAAAAAAAAAAAAAAAAAAAAAAAAAAAAAAAAAAAAAAAAAAAAAAAAAAAA"
+			"AAAAAAAAAAAAAAAAAAAAAAAAAAAAAAAAAAAAAAAAAAAAAAAAAAAAAAAAAAAAAAAAAAAAAAAAAAAA"
+			"AAAAAAAAAAAAAAAAAAAAAAAAAAAAAAAAAAAAAAAAAAAAAAAAAAAAAAAAAAAAAAAAAAAAAAAAAAAA"
+			"AAAAAAAAAAAAAAAAAAAAAAAAAAAAAAAAAAAAAAAAAAAAAAAAAAAAAAAAAAAAAAAAAAAAAAAAAAAA"
+			"AAAAAAAAAAAAAAAAAAAAAAAAAAAAAAAAAAAAAAAAAAAAAAAAAAAAAAAAAAAAAAAAAAAAAAAAAAAA"
+			"AAAAAAAAAAAAAAAAAAAAAAAAAAAAAAAAAAAAAAAAAAAAAAAAAAAAAAAAAAAAAAAAAAAAAAAAAAAA"
+			"AAAAAAAAAAAAAAAAAAAAAAAAAAAAAAAAAAAAAAAAAAAAAAAAAAAAAAAAAAAAAAAAAAAAAAAAAAAA"
+			"AAAAAAAAAAAAAAAAAAAAAAAAAAAAAAAAAAAAAAAAAAAAAAAAAAAAAAAAAAAAAAAAAAAAAAAAAAAA"
+			"AAAAAAAAAAAAAAAAAAAAAAAAAAAAAAAAAAAAAAAAAAAAAAAAAAAAAAAAAAAAAAAAAAAAAAAAAAAA"
+			"AAAAAAAAAAAAAAAAAAAAAAAAAAAAAAAAAAAAAAAAAAAAAAAAAAAAAAAAAAAAAAAAAAAAAAAAAAAA"
+			"AAAAAAAAAAAAAAAAAAAAAAAAAAAAAAAAAAAAAAAAAAAAAAAAAAAAAAAAAAAAAAAAAAAAAAAAAAAA"
+			"AAAAAAAAAAAAAAAAAAAAAAAAAAAAAAAAAAAAAAAAAAAAAAAAAAAAAAAAAAAAAAAAAAAAAAAAAAAA"
+			"AAAAAAAAAAAAAAAAAAAAAAAAAAAAAAAAAAAAAAAAAAAAAAAAAAAAAAAAAAAAAAAAAAAAAAAAAAAA"
+			"AAAAAAAAAAAAAAAAAAAAAAAAAAAAAAAAAAAAAAAAAAAAAAAAAAAAAAAAAAAAAAAAAAAAAAAAAAAA"
+			"AAAAAAAAAAAAAAAAAAAAAAAAAAAAAAAAAAAAAAAAAAAAAAAAAA=="
 		)
 	)
@@
 			)
 		)
+		(property "PN" "ERA-3AEB112V"
+			(at 166.37 96.52 90)
+			(effects
+				(font
+					(size 1.27 1.27)
+				)
+				(hide yes)
+			)
+		)
 		(pin "1"
 		)
@@
 			)
 		)
+		(property "PN" "ERA-3AEB112V"
+			(at 68.58 77.47 0)
+			(effects
+				(font
+					(size 1.27 1.27)
+				)
+				(hide yes)
+			)
+		)
 		(pin "1"
 		)
@@
 			)
 		)
+		(property "PN" "C0603X682F5GECTU"
+			(at 53.34 99.06 0)
+			(effects
+				(font
+					(size 1.27 1.27)
+				)
+				(hide yes)
+			)
+		)
 		(pin "2"
 		)
@@
 			)
 		)
+		(property "PN" "GCM1885C2A102FA16D"
+			(at 85.09 123.19 0)
+			(effects
+				(font
+					(size 1.27 1.27)
+				)
+				(hide yes)
+			)
+		)
 		(pin "2"
 		)
@@
 			)
 		)
+		(property "PN" "ERA-3AEB112V"
+			(at 40.64 96.52 90)
+			(effects
+				(font
+					(size 1.27 1.27)
+				)
+				(hide yes)
+			)
+		)
 		(pin "1"
 		)
@@
 			)
 		)
+		(property "PN" "ERA-3AEB121V"
+			(at 223.52 101.6 90)
+			(effects
+				(font
+					(size 1.27 1.27)
+				)
+				(hide yes)
+			)
+		)
 		(pin "1"
 		)
@@
 			)
 		)
+		(property "PN" "OPA1637DGKR"
+			(at 196.85 99.06 0)
+			(effects
+				(font
+					(size 1.27 1.27)
+				)
+				(hide yes)
+			)
+		)
 		(pin "6"
 		)
@@
 			)
 		)
+		(property "PN" "GCM1885C2A102FA16D"
+			(at 85.09 77.47 0)
+			(effects
+				(font
+					(size 1.27 1.27)
+				)
+				(hide yes)
+			)
+		)
 		(pin "2"
 		)
@@
 			)
 		)
+		(property "PN" "GCJ188R71H104KA12D"
+			(at 106.68 82.55 0)
+			(effects
+				(font
+					(size 1.27 1.27)
+				)
+				(hide yes)
+			)
+		)
 		(pin "2"
 		)
@@
 			)
 		)
+		(property "PN" "GRM2195C2A393GE01J"
+			(at 142.24 99.06 0)
+			(effects
+				(font
+					(size 1.27 1.27)
+				)
+				(hide yes)
+			)
+		)
 		(pin "2"
 		)
@@
 			)
 		)
+		(property "PN" "GCJ188R71H104KA12D"
+			(at 201.93 82.55 0)
+			(effects
+				(font
+					(size 1.27 1.27)
+				)
+				(hide yes)
+			)
+		)
 		(pin "2"
 		)
@@
 			)
 		)
+		(property "PN" "ERA-3AEB561V"
+			(at 77.47 96.52 90)
+			(effects
+				(font
+					(size 1.27 1.27)
+				)
+				(hide yes)
+			)
+		)
 		(pin "1"
 		)
@@
 			)
 		)
+		(property "PN" "ERA-3AEB112V"
+			(at 173.99 77.47 0)
+			(effects
+				(font
+					(size 1.27 1.27)
+				)
+				(hide yes)
+			)
+		)
 		(pin "1"
 		)
@@
 			)
 		)
+		(property "PN" "ERA-3AEB112V"
+			(at 166.37 101.6 90)
+			(effects
+				(font
+					(size 1.27 1.27)
+				)
+				(hide yes)
+			)
+		)
 		(pin "1"
 		)
@@
 			)
 		)
+		(property "PN" "ERA-3AEB112V"
+			(at 68.58 123.19 0)
+			(effects
+				(font
+					(size 1.27 1.27)
+				)
+				(hide yes)
+			)
+		)
 		(pin "1"
 		)
@@
 			)
 		)
+		(property "PN" "ERA-3AEB561V"
+			(at 77.47 101.6 90)
+			(effects
+				(font
+					(size 1.27 1.27)
+				)
+				(hide yes)
+			)
+		)
 		(pin "1"
 		)
@@
 		(property "Description" "Resistor, small symbol"
 			(at 129.54 101.6 0)
+			(effects
+				(font
+					(size 1.27 1.27)
+				)
+				(hide yes)
+			)
+		)
+		(property "PN" "ERA-3AEB470V"
+			(at 129.54 101.6 90)
 			(effects
 				(font
@@
 			)
 		)
+		(property "PN" "ERA-3AEB470V"
+			(at 129.54 96.52 90)
+			(effects
+				(font
+					(size 1.27 1.27)
+				)
+				(hide yes)
+			)
+		)
 		(pin "1"
 		)
@@
 			)
 		)
+		(property "PN" "ERA-3AEB112V"
+			(at 173.99 123.19 0)
+			(effects
+				(font
+					(size 1.27 1.27)
+				)
+				(hide yes)
+			)
+		)
 		(pin "1"
 		)
@@
 			)
 		)
+		(property "PN" "OPA1637DGKR"
+			(at 101.6 99.06 0)
+			(effects
+				(font
+					(size 1.27 1.27)
+				)
+				(hide yes)
+			)
+		)
 		(pin "6"
 		)
@@
 		(property "Description" "Resistor, small symbol"
 			(at 40.64 101.6 0)
+			(effects
+				(font
+					(size 1.27 1.27)
+				)
+				(hide yes)
+			)
+		)
+		(property "PN" "ERA-3AEB112V"
+			(at 40.64 101.6 90)
 			(effects
 				(font
@@
 			(effects
 				(font
+					(size 1.27 1.27)
+				)
+				(hide yes)
+			)
+		)
+		(property "PN" "ERA-3AEB121V"
+			(at 223.52 96.52 90)
+			(effects
+				(font
