File: amp.kicad_sch (KiCad schematic)
At the start: 17 parts, among them J17 ACJS-MV35-3, U11 OPA1637

Commit message: WIP layout
Other:
- note added: "For unused inputs: "The second form of termination is to connect the positive (+) pin and negative (-) pins together and terminating these to AGNDAD with 0.001-μF to 1-μF capacitors. This option applies to unused pins with channels that are configured in differential mode" AWL: load shunt across final outout cap and then layout is such that a small jumper or shunt can be placed from this node to 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"
- note added: "pin 3 should be + pin 4 should be - pin 1 is shield (gnd) flipping the connections at the input compensates for the amp inversion"
- note removed: "connectors: amphenol ACJS-MV35-3 same sky SJ3-35053A"
- note removed: "wire up based on chosen connector"

Commit message: DONE. now exporting gerbers
Parts:
- C41: footprint Capacitor_SMD:C_0603_1608Metric -> Capacitor_SMD:C_0805_2012Metric
- U11: footprint Package_SO:SOIC-8_3.9x4.9mm_P1.27mm -> Package_SO:MSOP-8_3x3mm_P0.65mm
