File: digital_input_buffer.kicad_sch (KiCad schematic)
At the start: 8 parts, among them J9 Conn_Coaxial, U2 74LVC1G17

Commit message: redoing file add
Parts:
- renumbered C13 to C17, C14 to C18, R26 to R22, R27 to R23, R28 to R24
Changed lines of the file:
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@@
 		(dnp no)
 		(fields_autoplaced yes)
-		(property "Reference" "#PWR033"
+		(property "Reference" "#PWR037"
 			(at 167.64 87.63 0)
 			(effects
@@
 			(project "pcm3168a_euro1"
 				(path "/afe1fbe1-30b6-4eb7-94cf-5d2700d51271/1278d92a-e870-421c-8ab2-98a46892c829"
-					(reference "#PWR033")
-					(unit 1)
-				)
-				(path "/afe1fbe1-30b6-4eb7-94cf-5d2700d51271/c889fde3-e058-4b42-9958-89d0b807b204"
-					(reference "#PWR066")
-					(unit 1)
-				)
-				(path "/afe1fbe1-30b6-4eb7-94cf-5d2700d51271/f5984572-3a10-4c6c-8f40-83f484c9a466"
-					(reference "#PWR042")
+					(reference "#PWR037")
+					(unit 1)
+				)
+				(path "/afe1fbe1-30b6-4eb7-94cf-5d2700d51271/c889fde3-e058-4b42-9958-89d0b807b204"
+					(reference "#PWR070")
+					(unit 1)
+				)
+				(path "/afe1fbe1-30b6-4eb7-94cf-5d2700d51271/f5984572-3a10-4c6c-8f40-83f484c9a466"
+					(reference "#PWR046")
 					(unit 1)
 				)
@@
 		(dnp no)
 		(fields_autoplaced yes)
-		(property "Reference" "C14"
+		(property "Reference" "C18"
 			(at 170.561 76.2578 0)
 			(effects
@@
 			(project "pcm3168a_euro1"
 				(path "/afe1fbe1-30b6-4eb7-94cf-5d2700d51271/1278d92a-e870-421c-8ab2-98a46892c829"
-					(reference "C14")
-					(unit 1)
-				)
-				(path "/afe1fbe1-30b6-4eb7-94cf-5d2700d51271/c889fde3-e058-4b42-9958-89d0b807b204"
-					(reference "C28")
-					(unit 1)
-				)
-				(path "/afe1fbe1-30b6-4eb7-94cf-5d2700d51271/f5984572-3a10-4c6c-8f40-83f484c9a466"
 					(reference "C18")
+					(unit 1)
+				)
+				(path "/afe1fbe1-30b6-4eb7-94cf-5d2700d51271/c889fde3-e058-4b42-9958-89d0b807b204"
+					(reference "C32")
+					(unit 1)
+				)
+				(path "/afe1fbe1-30b6-4eb7-94cf-5d2700d51271/f5984572-3a10-4c6c-8f40-83f484c9a466"
+					(reference "C22")
 					(unit 1)
 				)
@@
 		(dnp yes)
 		(fields_autoplaced yes)
-		(property "Reference" "C13"
+		(property "Reference" "C17"
 			(at 144.5641 97.8541 0)
 			(effects
@@
 			(project "pcm3168a_euro1"
 				(path "/afe1fbe1-30b6-4eb7-94cf-5d2700d51271/1278d92a-e870-421c-8ab2-98a46892c829"
-					(reference "C13")
-					(unit 1)
-				)
-				(path "/afe1fbe1-30b6-4eb7-94cf-5d2700d51271/c889fde3-e058-4b42-9958-89d0b807b204"
-					(reference "C27")
-					(unit 1)
-				)
-				(path "/afe1fbe1-30b6-4eb7-94cf-5d2700d51271/f5984572-3a10-4c6c-8f40-83f484c9a466"
 					(reference "C17")
+					(unit 1)
+				)
+				(path "/afe1fbe1-30b6-4eb7-94cf-5d2700d51271/c889fde3-e058-4b42-9958-89d0b807b204"
+					(reference "C31")
+					(unit 1)
+				)
+				(path "/afe1fbe1-30b6-4eb7-94cf-5d2700d51271/f5984572-3a10-4c6c-8f40-83f484c9a466"
+					(reference "C21")
 					(unit 1)
 				)
@@
 		(dnp yes)
 		(fields_autoplaced yes)
-		(property "Reference" "R27"
+		(property "Reference" "R23"
 			(at 131.0386 97.8478 0)
 			(effects
@@
 			(project "pcm3168a_euro1"
 				(path "/afe1fbe1-30b6-4eb7-94cf-5d2700d51271/1278d92a-e870-421c-8ab2-98a46892c829"
-					(reference "R27")
-					(unit 1)
-				)
-				(path "/afe1fbe1-30b6-4eb7-94cf-5d2700d51271/c889fde3-e058-4b42-9958-89d0b807b204"
-					(reference "R47")
-					(unit 1)
-				)
-				(path "/afe1fbe1-30b6-4eb7-94cf-5d2700d51271/f5984572-3a10-4c6c-8f40-83f484c9a466"
-					(reference "R33")
+					(reference "R23")
+					(unit 1)
+				)
+				(path "/afe1fbe1-30b6-4eb7-94cf-5d2700d51271/c889fde3-e058-4b42-9958-89d0b807b204"
+					(reference "R43")
+					(unit 1)
+				)
+				(path "/afe1fbe1-30b6-4eb7-94cf-5d2700d51271/f5984572-3a10-4c6c-8f40-83f484c9a466"
+					(reference "R29")
 					(unit 1)
 				)
@@
 		(dnp no)
 		(fields_autoplaced yes)
-		(property "Reference" "R26"
+		(property "Reference" "R22"
 			(at 123.19 86.7633 90)
 			(effects
@@
 			(project "pcm3168a_euro1"
 				(path "/afe1fbe1-30b6-4eb7-94cf-5d2700d51271/1278d92a-e870-421c-8ab2-98a46892c829"
-					(reference "R26")
-					(unit 1)
-				)
-				(path "/afe1fbe1-30b6-4eb7-94cf-5d2700d51271/c889fde3-e058-4b42-9958-89d0b807b204"
-					(reference "R46")
-					(unit 1)
-				)
-				(path "/afe1fbe1-30b6-4eb7-94cf-5d2700d51271/f5984572-3a10-4c6c-8f40-83f484c9a466"
-					(reference "R32")
+					(reference "R22")
+					(unit 1)
+				)
+				(path "/afe1fbe1-30b6-4eb7-94cf-5d2700d51271/c889fde3-e058-4b42-9958-89d0b807b204"
+					(reference "R42")
+					(unit 1)
+				)
+				(path "/afe1fbe1-30b6-4eb7-94cf-5d2700d51271/f5984572-3a10-4c6c-8f40-83f484c9a466"
+					(reference "R28")
 					(unit 1)
 				)
@@
 		(dnp no)
 		(fields_autoplaced yes)
-		(property "Reference" "#PWR031"
+		(property "Reference" "#PWR035"
 			(at 161.29 76.2 0)
 			(effects
@@
 			(project "pcm3168a_euro1"
 				(path "/afe1fbe1-30b6-4eb7-94cf-5d2700d51271/1278d92a-e870-421c-8ab2-98a46892c829"
-					(reference "#PWR031")
-					(unit 1)
-				)
-				(path "/afe1fbe1-30b6-4eb7-94cf-5d2700d51271/c889fde3-e058-4b42-9958-89d0b807b204"
-					(reference "#PWR064")
-					(unit 1)
-				)
-				(path "/afe1fbe1-30b6-4eb7-94cf-5d2700d51271/f5984572-3a10-4c6c-8f40-83f484c9a466"
-					(reference "#PWR040")
+					(reference "#PWR035")
+					(unit 1)
+				)
+				(path "/afe1fbe1-30b6-4eb7-94cf-5d2700d51271/c889fde3-e058-4b42-9958-89d0b807b204"
+					(reference "#PWR068")
+					(unit 1)
+				)
+				(path "/afe1fbe1-30b6-4eb7-94cf-5d2700d51271/f5984572-3a10-4c6c-8f40-83f484c9a466"
+					(reference "#PWR044")
 					(unit 1)
 				)
@@
 		(dnp no)
 		(fields_autoplaced yes)
-		(property "Reference" "#PWR030"
+		(property "Reference" "#PWR034"
 			(at 109.22 113.03 0)
 			(effects
@@
 			(project "pcm3168a_euro1"
 				(path "/afe1fbe1-30b6-4eb7-94cf-5d2700d51271/1278d92a-e870-421c-8ab2-98a46892c829"
-					(reference "#PWR030")
-					(unit 1)
-				)
-				(path "/afe1fbe1-30b6-4eb7-94cf-5d2700d51271/c889fde3-e058-4b42-9958-89d0b807b204"
-					(reference "#PWR063")
-					(unit 1)
-				)
-				(path "/afe1fbe1-30b6-4eb7-94cf-5d2700d51271/f5984572-3a10-4c6c-8f40-83f484c9a466"
-					(reference "#PWR039")
+					(reference "#PWR034")
+					(unit 1)
+				)
+				(path "/afe1fbe1-30b6-4eb7-94cf-5d2700d51271/c889fde3-e058-4b42-9958-89d0b807b204"
+					(reference "#PWR067")
+					(unit 1)
+				)
+				(path "/afe1fbe1-30b6-4eb7-94cf-5d2700d51271/f5984572-3a10-4c6c-8f40-83f484c9a466"
+					(reference "#PWR043")
 					(unit 1)
 				)
@@
 		(dnp no)
 		(fields_autoplaced yes)
-		(property "Reference" "#PWR032"
+		(property "Reference" "#PWR036"
 			(at 161.29 114.3 0)
 			(effects
@@
 			(project "pcm3168a_euro1"
 				(path "/afe1fbe1-30b6-4eb7-94cf-5d2700d51271/1278d92a-e870-421c-8ab2-98a46892c829"
-					(reference "#PWR032")
-					(unit 1)
-				)
-				(path "/afe1fbe1-30b6-4eb7-94cf-5d2700d51271/c889fde3-e058-4b42-9958-89d0b807b204"
-					(reference "#PWR065")
-					(unit 1)
-				)
-				(path "/afe1fbe1-30b6-4eb7-94cf-5d2700d51271/f5984572-3a10-4c6c-8f40-83f484c9a466"
-					(reference "#PWR041")
+					(reference "#PWR036")
+					(unit 1)
+				)
+				(path "/afe1fbe1-30b6-4eb7-94cf-5d2700d51271/c889fde3-e058-4b42-9958-89d0b807b204"
+					(reference "#PWR069")
+					(unit 1)
+				)
+				(path "/afe1fbe1-30b6-4eb7-94cf-5d2700d51271/f5984572-3a10-4c6c-8f40-83f484c9a466"
+					(reference "#PWR045")
 					(unit 1)
 				)
@@
 		(dnp no)
 		(fields_autoplaced yes)
-		(property "Reference" "R28"
+		(property "Reference" "R24"
 			(at 185.42 86.7633 90)
 			(effects
@@
 			(project "pcm3168a_euro1"
 				(path "/afe1fbe1-30b6-4eb7-94cf-5d2700d51271/1278d92a-e870-421c-8ab2-98a46892c829"
-					(reference "R28")
-					(unit 1)
-				)
-				(path "/afe1fbe1-30b6-4eb7-94cf-5d2700d51271/c889fde3-e058-4b42-9958-89d0b807b204"
-					(reference "R48")
-					(unit 1)
-				)
-				(path "/afe1fbe1-30b6-4eb7-94cf-5d2700d51271/f5984572-3a10-4c6c-8f40-83f484c9a466"
-					(reference "R34")
-					(unit 1)
-				)
+					(reference "R24")
+					(unit 1)
+				)
+				(path "/afe1fbe1-30b6-4eb7-94cf-5d2700d51271/c889fde3-e058-4b42-9958-89d0b807b204"
+					(reference "R44")
+					(unit 1)
+				)
+				(path "/afe1fbe1-30b6-4eb7-94cf-5d2700d51271/f5984572-3a10-4c6c-8f40-83f484c9a466"
+					(reference "R30")
+					(unit 1)
+				)

Commit message: WIP need to fix OPA1637 footprint
Parts:
- J9: footprint Connector_Coaxial:SMA_Amphenol_901-144_Vertical -> pcm3168a_euro1:SMA_Amphenol_901-144_Vertical_awl1
Changed lines of the file:
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@@
 			)
 		)
-		(property "Footprint" "Connector_Coaxial:SMA_Amphenol_901-144_Vertical"
+		(property "Footprint" "pcm3168a_euro1:SMA_Amphenol_901-144_Vertical_awl1"
 			(at 109.22 91.44 0)
 			(effects

Commit message: added part numbers
Parts:
- C18: PN (none) -> GCJ188R71H104KA12D
- D1: PN (none) -> SMF5.0A
- R22: PN (none) -> CRCW06030000Z0EA
- R24: PN (none) -> CRCW060322R0FKEAC
- U2: PN (none) -> SN74LVC1G17DBVR
Changed lines of the file:
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@@
+			)
+		)
+		(property "PN" "GCJ188R71H104KA12D"
+			(at 167.64 77.47 0)
+			(effects
+				(font
+					(size 1.27 1.27)
+				)
+				(hide yes)
 			)
 		)
@@
 			)
 		)
+		(property "PN" "CRCW06030000Z0EA"
+			(at 123.19 91.44 90)
+			(effects
+				(font
+					(size 1.27 1.27)
+				)
+				(hide yes)
+			)
+		)
 		(pin "2"
 		)
@@
 			)
 		)
+		(property "PN" "SN74LVC1G17DBVR"
+			(at 166.37 91.44 0)
+			(effects
+				(font
+					(size 1.27 1.27)
+				)
+				(hide yes)
+			)
+		)
 		(pin "2"
 		)
@@
 			)
 		)
+		(property "PN" "CRCW060322R0FKEAC"
+			(at 185.42 91.44 90)
+			(effects
+				(font
+					(size 1.27 1.27)
+				)
+				(hide yes)
+			)
+		)
 		(pin "2"
 		)
@@
 			(effects
 				(font
+					(size 1.27 1.27)
+				)
+				(hide yes)
+			)
+		)
+		(property "PN" "SMF5.0A"
+			(at 116.84 97.79 90)
+			(effects
+				(font
