File: digital_output_buffer.kicad_sch (KiCad schematic)
At the start: 7 parts, among them J10 Conn_Coaxial, U3 74LVC1G17

Commit message: redoing file add
Parts:
- renumbered C15 to C19, C16 to C20, R29 to R25, R30 to R26, R31 to R27

Commit message: WIP need to fix OPA1637 footprint
Parts:
- J10: footprint Connector_Coaxial:SMA_Amphenol_901-144_Vertical -> pcm3168a_euro1:SMA_Amphenol_901-144_Vertical_awl1
Changed lines of the file:
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@@
 			)
 		)
-		(property "Footprint" "Connector_Coaxial:SMA_Amphenol_901-144_Vertical"
+		(property "Footprint" "pcm3168a_euro1:SMA_Amphenol_901-144_Vertical_awl1"
 			(at 199.39 99.06 0)
 			(effects

Commit message: added part numbers
Parts:
- C20: PN (none) -> GCJ188R71H104KA12D
- R25: PN (none) -> CRCW06030000Z0EA
- R27: PN (none) -> CRCW060322R0FKEAC
- U3: PN (none) -> SN74LVC1G17DBVR
Changed lines of the file:
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@@
+			)
+		)
+		(property "PN" "SN74LVC1G17DBVR"
+			(at 163.83 99.06 0)
+			(effects
+				(font
+					(size 1.27 1.27)
+				)
+				(hide yes)
 			)
 		)
@@
 			)
 		)
+		(property "PN" "CRCW06030000Z0EA"
+			(at 120.65 99.06 90)
+			(effects
+				(font
+					(size 1.27 1.27)
+				)
+				(hide yes)
+			)
+		)
 		(pin "2"
 		)
@@
 			)
 		)
+		(property "PN" "GCJ188R71H104KA12D"
+			(at 165.1 85.09 0)
+			(effects
+				(font
+					(size 1.27 1.27)
+				)
+				(hide yes)
+			)
+		)
 		(pin "1"
 		)
@@
 			(effects
 				(font
+					(size 1.27 1.27)
+				)
+				(hide yes)
+			)
+		)
+		(property "PN" "CRCW060322R0FKEAC"
+			(at 182.88 99.06 90)
+			(effects
+				(font
