File: pcm3168a_euro1.kicad_sch (KiCad schematic)
At the start: 47 parts, among them J8 Conn_01x02_Pin, U1 PCM3168APAPR

Commit message: DONE. now exporting gerbers
Other:
- note added: "TODO - fix footprint for 39n caps - check footprint for 6.8n caps"
- note removed: "- fix OPA1637 footprint - double check IC footprints, leave note on schematic for checked footprint - tant polarity silkscreen"
- note removed: "FOOTPRINT OK"
- moved on the sheet: C1, C10, C11, C12, C120, C121, C13, C14, C15, C16, C2, C3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

Commit message: added part numbers
Parts:
- C1, C11, C12, C13, C14, C15, C16, C2, C7, C8: PN (none) -> GRM31CR71E106KA12L
- C10, C3, C4, C5, C6, C9: PN (none) -> GCM188R71C105KA64J
- C120, C121: PN (none) -> GCJ188R71H104KA12D
- J8: PN (none) -> 61300211121
- R1, R11, R13, R14, R16: PN (none) -> CRCW0603220KFKEAC
- R19: PN (none) -> ERA-3AEB472V
- R20, R60, R90: PN (none) -> CRCW060322R0FKEAC
- R3, R4, R5, R6, R7, R8: PN (none) -> CRCW06030000Z0EA
- U1: PN (none) -> PCM3168APAP
