File: power.kicad_sch (KiCad schematic)
At the start: 21 parts, among them J18 Conn_02x08_Odd_Even, J19 Conn_Coaxial, U12 TLV1117-33

Commit message: DONE. now exporting gerbers
Other:
- note removed: "FOOTPRINT OK"
- moved on the sheet: C42, C43, C44, C45, C46, C47, C48, C49, C50, C59, C62, C65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

Commit message: added part numbers
Parts:
- C42, C45, C46, C59: PN (none) -> UES1C470MPM1TD
- D3: PN (none) -> WP710A10ID
- J18: PN (none) -> PPPC082LFBN-RC
- L1, L2: PN (none) -> BLM18KG601SN1D
- R139: PN (none) -> ERA-3AEB472V
- R56, R57: PN (none) -> CRCW06030000Z0EA
- U12: PN (none) -> TLV1117-33IDCYR
Changed lines of the file:
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@@
 			"AAAAAAAAAAAAAAAAAAAAAAAAAAAAAAAAAACAAAAAAAAAAAAAAAAAAAAAAAAAAAAAAAAAAAAAAEAO"
 			"XOcZcAAAQQEAAAAAAACgqRV1qFcAAFAECHWoVwAAAJqRdahXAAAQaRR1qFcAALCdFXWoVwAAAAAA"
-			"AAAAAABAAAAAAAAAAEAAAAAAAAAAmayAD61XAAAAAAAAAAAAAGAICA=="
+			"AAAAAABAAAAAAAAAAEAAAAAAAAAAmayAD61XAAAAAAAAAAAAAGAICAAAAAAAAAAAAAAAAAAAAAAA"
+			"AAAAAAAAAAAAAAAAAAAAAAAAAAAAAAAAAAAAAAAAAAAAAAAAAAAAAAAAAAAAAAAAAAAAAAAAAAAA"
+			"AAAAAAAAAAAAAAAAAAAAAAAAAAAAAAAAAAAAAAAAAAAAAAAAAAAAAAAAAAAAAAAAAAAAAAAAAAAA"
+			"AAAAAAAAAAAAAAAAAAAAAAAAAAAAAAAAAAAAAAAAAAAAAAAAAAAAAAAAAAAAAAAAAAAAAAAAAAAA"
+			"AAAAAAAAAAAAAAAAAAAAAAAAAAAAAAAAAAAAAAAAAAAAAAAAAAAAAAAAAAAAAAAAAAAAAAAAAAAA"
+			"AAAAAAAAAAAAAAAAAAAAAAAAAAAAAAAAAAAAAAAAAAAAAAAAAAAAAAAAAAAAAAAAAAAAAAAAAAAA"
+			"AAAAAAAAAAAAAAAAAAAAAAAAAAAAAAAAAAAAAAAAAAAAAAAAAAAAAAAAAAAAAAAAAAAAAAAAAAAA"
+			"AAAAAAAAAAAAAAAAAAAAAAAAAAAAAAAAAAAAAAAAAAAAAAAAAAAAAAAAAAAAAAAAAAAAAAAAAAAA"
+			"AAAAAAAAAAAAAAAAAAAAAAAAAAAAAAAAAAAAAAAAAAAAAAAAAAAAAAAAAAAAAAAAAAAAAAAAAAAA"
+			"AAAAAAAAAAAAAAAAAAAAAAAAAAAAAAAAAAAAAAAAAAAAAAAAAAAAAAAAAAAAAAAAAAAAAAAAAAAA"
+			"AAAAAAAAAAAAAAAAAAAAAAAAAAAAAAAAAAAAAAAAAAAAAAAAAAAAAAAAAAAAAAAAAAAAAAAAAAAA"
+			"AAAAAAAAAAAAAAAAAAAAAAAAAAAAAAAAAAAAAAAAAAAAAAAAAAAAAAAAAAAAAAAAAAAAAAAAAAAA"
+			"AAAAAAAAAAAAAAAAAAAAAAAAAAAAAAAAAAAAAAAAAAAAAAAAAAAAAAAAAAAAAAAAAAAAAAAAAAAA"
+			"AAAAAAAAAAAAAAAAAAAAAAAAAAAAAAAAAAAAAAAAAAAAAAAAAAAAAAAAAAAAAAAAAAAAAAAAAAAA"
+			"AAAAAAAAAAAAAAAAAAAAAAAAAAAAAAAAAAAAAAAAAAAAAAAAAAAAAAAAAAAAAAAAAAAAAAAAAAAA"
+			"AAAAAAAAAAAAAAAAAAAAAAAAAAAAAAAAAAAAAAAAAAAAAAAAAAAAAAAAAAAAAAAAAAAAAAAAAAAA"
+			"AAAAAAAAAAAAAAAAAAAAAAAAAAAAAAAAAAAAAAAAAAAAAAAAAAAAAAAAAAAAAAAAAAAAAAAAAAAA"
+			"AAAAAAAAAAAAAAAAAAAAAAAAAAAAAAAAAAAAAAAAAAAAAAAAAAAAAAAAAAAAAAAAAAAAAAAAAAAA"
+			"AAAAAAAAAAAAAAAAAAAAAAAAAAAAAAAAAAAAAAAAAAAAAAAAAAAAAA=="
 		)
 	)
@@
 			"AOCh764ZcAAAIL9udKhXAAAAAAAA8pRxv6cBnD45CwQ+FQ1vv41BmD6txEs+wdR6v9A2ID547/49"
 			"0iccQY7vUcHkvy0/dSkcQV/wUcFwni4/6QccQTG3UsHkvy0/IdN6v1FeID4j8v49AAAAAAAAAAAA"
+			"AAAAaQAAADUAAABOAAAAUwAAAHMAAAB5AAAARgAAAGkAAABoAAAAcwAAAHQAAAArAAAANwAAAFAA"
+			"AAAvAAAAVgAAAHoAAAAyAAAAUQAAAEIAAABZAAAATAAAADEAAAAyAAAAVQAAAE0AAAAyAAAAQgAA"
+			"AGEAAAA2AAAAdQAAAFIAAABYAAAAaQAAAGQAAABJAAAAQgAAAGcAAAB6AAAARAAAAEoAAABTAAAA"
+			"QQAAAEIAAABXAAAAaQAAAGEAAAB4AAAAKwAAAHEAAAA5AAAAYgAAAGUAAAArAAAASQAAADgAAABj"
+			"AAAAUAAAAEcAAABsAAAAcQAAAEwAAAA4AAAAOAAAADgAAABlAAAAZgAAAGgAAABHAAAARgAAADQA"
+			"AAAwAAAAbQAAADcAAABYAAAARQAAAGIAAABLAAAAMgAAAHQAAAAvAAAATwAAAHQAAABGAAAAcgAA"
+			"AHAAAAArAAAASAAAAFIAAAAwAAAAZgAAAG4AAABuAAAAcQAAAHEAAABYAAAATQAAAHkAAABxAAAA"
+			"UQAAAFkAAABBAAAAQQAAAHEAAABHAAAAVQAAAHAAAABxAAAAZwAAAG8AAABFAAAAcwAAAHkAAABR"
+			"AAAAeQAAADUAAABnAAAAZQAAAG8AAAA1AAAAdwAAAEgAAABuAAAAOAAAAHYAAABQAAAAUAAAAHcA"
+			"AAB6AAAAdQAAADMAAAB2AAAASAAAAC8AAAA0AAAAZQAAAC8AAABMAAAARAAAAEgAAAB4AAAAYgAA"
+			"ACsAAAA4AAAAMwAAADgAAAAyAAAAcgAAADEAAAA0AAAAZAAAAGgAAABKAAAAMgAAAFQAAABmAAAA"
+			"QgAAAHYAAABXAAAANgAAADAAAABsAAAAQwAAACsAAABQAAAAWQAAADIAAABiAAAANwAAAGQAAABs"
+			"AAAAcgAAADQAAABmAAAAMgAAAEQAAAAxAAAAZwAAACsAAABKAAAAOAAAAE8AAABBAAAAVgAAAHkA"
+			"AABxAAAANAAAAFcAAABNAAAAUwAAADUAAAAvAAAARgAAAFAAAABsAAAASAAAAFQAAAAvAAAAMAAA"
+			"ADkAAABSAAAAOAAAAGMAAABzAAAASAAAAC8AAAArAAAAWgAAAC8AAABiAAAARgAAAGwAAAA4AAAA"
+			"SgAAADIAAAA2AAAAUAAAAHAAAABaAAAAbQAAAHMAAAA5AAAAVAAAADIAAAB3AAAAWgAAAFYAAABq"
+			"AAAAZQAAAGYAAABxAAAAWAAAAE4AAABmAAAAWgAAAFEAAABZAAAATgAAAHYAAABiAAAAdgAAAEYA"
+			"AABLAAAARgAAAGUAAABrAAAARwAAAE8AAABtAAAAaQAAAEkAAABJAAAARQAAAEMAAABtAAAAUwAA"
 			"AA=="
 		)
@@
 			)
 		)
+		(property "PN" "BLM18KG601SN1D"
+			(at 168.91 73.66 90)
+			(effects
+				(font
+					(size 1.27 1.27)
+				)
+				(hide yes)
+			)
+		)
 		(pin "2"
 		)
@@
 			)
 		)
+		(property "PN" "BLM18KG601SN1D"
+			(at 168.91 44.45 90)
+			(effects
+				(font
+					(size 1.27 1.27)
+				)
+				(hide yes)
+			)
+		)
 		(pin "2"
 		)
@@
 			)
 		)
+		(property "PN" "CRCW06030000Z0EA"
+			(at 128.27 44.45 90)
+			(effects
+				(font
+					(size 1.27 1.27)
+				)
+				(hide yes)
+			)
+		)
 		(pin "2"
 		)
@@
 			)
 		)
+		(property "PN" "UES1C470MPM1TD"
+			(at 226.06 80.01 0)
+			(effects
+				(font
+					(size 1.27 1.27)
+				)
+				(hide yes)
+			)
+		)
 		(pin "1"
 		)
@@
 			)
 		)
+		(property "PN" "TLV1117-33IDCYR"
+			(at 212.09 73.66 0)
+			(effects
+				(font
+					(size 1.27 1.27)
+				)
+				(hide yes)
+			)
+		)
 		(pin "2"
 		)
@@
 			)
 		)
+		(property "PN" "UES1C470MPM1TD"
+			(at 177.8 50.8 0)
+			(effects
+				(font
+					(size 1.27 1.27)
+				)
+				(hide yes)
+			)
+		)
 		(pin "1"
 		)
@@
 			)
 		)
+		(property "PN" "PPPC082LFBN-RC"
+			(at 82.55 49.53 0)
+			(effects
+				(font
+					(size 1.27 1.27)
+				)
+				(hide yes)
+			)
+		)
 		(pin "12"
 		)
@@
 			)
 		)
+		(property "PN" "CRCW06030000Z0EA"
+			(at 138.43 36.83 90)
+			(effects
+				(font
+					(size 1.27 1.27)
+				)
+				(hide yes)
+			)
+		)
 		(pin "2"
 		)
@@
 			)
 		)
+		(property "PN" "UES1C470MPM1TD"
+			(at 146.05 50.8 0)
+			(effects
+				(font
+					(size 1.27 1.27)
+				)
+				(hide yes)
+			)
+		)
 		(pin "1"
 		)
@@
 			)
 		)
+		(property "PN" "UES1C470MPM1TD"
+			(at 177.8 80.01 0)
+			(effects
+				(font
+					(size 1.27 1.27)
+				)
+				(hide yes)
+			)
+		)
 		(pin "1"
 		)
@@
 			)
 		)
+		(property "PN" "WP710A10ID"
+			(at 261.62 80.01 90)
+			(effects
+				(font
+					(size 1.27 1.27)
+				)
+				(hide yes)
+			)
+		)
 		(pin "1"
 		)
@@
 			(effects
 				(font
+					(size 1.27 1.27)
+				)
+				(hide yes)
+			)
+		)
+		(property "PN" "ERA-3AEB472V"
+			(at 261.62 91.44 90)
+			(effects
+				(font
