File: tdm_b1/buffer.kicad_sch (KiCad schematic)
At the start: 5 parts, among them U6 74LVC1G17

Commit message: filled out part number for tdm_b1
Parts:
- C26: PN (none) -> GCJ188R71H104KA12D
- R36: PN (none) -> CRCW060333R0FKEAC
- U6: PN (none) -> SN74LVC1G17DBVR
Changed lines of the file:
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@@
+			)
+		)
+		(property "PN" "GCJ188R71H104KA12D"
+			(at 124.46 62.23 0)
+			(effects
+				(font
+					(size 1.27 1.27)
+				)
+				(hide yes)
 			)
 		)
@@
 			)
 		)
+		(property "PN" "CRCW060333R0FKEAC"
+			(at 142.24 76.2 90)
+			(effects
+				(font
+					(size 1.27 1.27)
+				)
+				(hide yes)
+			)
+		)
 		(pin "2"
 		)
@@
 			(at 123.19 76.2 0)
 			(effects
+				(font
+					(size 1.27 1.27)
+				)
+				(hide yes)
+			)
+		)
+		(property "PN" "SN74LVC1G17DBVR"
+			(at 123.19 76.2 0)
+			(effects
