File: tdm_b1/digital_output.kicad_sch (KiCad schematic)
At the start: 7 parts, among them J12 Conn_Coaxial, U5 74LVC1G17

Commit message: filled out part number for tdm_b1
Parts:
- C24: PN (none) -> GCJ188R71H104KA12D
- R31: PN (none) -> CRCW06030000Z0EA
- R33: PN (none) -> CRCW060333R0FKEAC
- U5: PN (none) -> SN74LVC1G17DBVR
Changed lines of the file:
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@@
+			)
+		)
+		(property "PN" "SN74LVC1G17DBVR"
+			(at 156.21 104.14 0)
+			(effects
+				(font
+					(size 1.27 1.27)
+				)
+				(hide yes)
 			)
 		)
@@
 			)
 		)
+		(property "PN" "CRCW06030000Z0EA"
+			(at 113.03 104.14 90)
+			(effects
+				(font
+					(size 1.27 1.27)
+				)
+				(hide yes)
+			)
+		)
 		(pin "2"
 		)
@@
 			)
 		)
+		(property "PN" "GCJ188R71H104KA12D"
+			(at 157.48 90.17 0)
+			(effects
+				(font
+					(size 1.27 1.27)
+				)
+				(hide yes)
+			)
+		)
 		(pin "1"
 		)
@@
 			(effects
 				(font
+					(size 1.27 1.27)
+				)
+				(hide yes)
+			)
+		)
+		(property "PN" "CRCW060333R0FKEAC"
+			(at 175.26 104.14 90)
+			(effects
+				(font
