File: tdm_b1/midi_in.kicad_sch (KiCad schematic)
At the start: 7 parts, among them J3 AudioJack3, U1 6N137

Commit message: filled out part number for tdm_b1
Parts:
- C28: PN (none) -> GCJ188R71H104KA12D
- D4: PN (none) -> 1N4148W
- J3: PN (none) -> SJ1-3523N
- R39: PN (none) -> CRCW0603220RFKEA
- R40: PN (none) -> CRCW0603470RFKEA
- R47: PN (none) -> CRCW06030000Z0EA
- U1: PN (none) -> 160-1791-ND
Changed lines of the file:
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@@
+			)
+		)
+		(property "PN" "1N4148W"
+			(at 132.08 101.6 90)
+			(effects
+				(font
+					(size 1.27 1.27)
+				)
+				(hide yes)
 			)
 		)
@@
 			)
 		)
+		(property "PN" "CRCW06030000Z0EA"
+			(at 111.76 113.03 0)
+			(effects
+				(font
+					(size 1.27 1.27)
+				)
+				(hide yes)
+			)
+		)
 		(pin "2"
 		)
@@
 			)
 		)
+		(property "PN" "GCJ188R71H104KA12D"
+			(at 137.16 86.36 0)
+			(effects
+				(font
+					(size 1.27 1.27)
+				)
+				(hide yes)
+			)
+		)
 		(pin "1"
 		)
@@
 			)
 		)
+		(property "PN" "CRCW0603470RFKEA"
+			(at 165.1 90.17 0)
+			(effects
+				(font
+					(size 1.27 1.27)
+				)
+				(hide yes)
+			)
+		)
 		(pin "2"
 		)
@@
 			)
 		)
+		(property "PN" "SJ1-3523N"
+			(at 102.87 97.79 0)
+			(effects
+				(font
+					(size 1.27 1.27)
+				)
+				(hide yes)
+			)
+		)
 		(pin "S"
 		)
@@
 			)
 		)
+		(property "PN" "160-1791-ND"
+			(at 147.32 100.33 0)
+			(effects
+				(font
+					(size 1.27 1.27)
+				)
+				(hide yes)
+			)
+		)
 		(pin "4"
 		)
@@
 			(effects
 				(font
+					(size 1.27 1.27)
+				)
+				(hide yes)
+			)
+		)
+		(property "PN" "CRCW0603220RFKEA"
+			(at 124.46 97.79 90)
+			(effects
+				(font
