File: tdm_b1/midi_out.kicad_sch (KiCad schematic)
At the start: 3 parts, among them J2 AudioJack3

Commit message: filled out part number for tdm_b1
Parts:
- J2: PN (none) -> SJ1-3523N
- R38: PN (none) -> CRCW06032K20FKEA
- R48: PN (none) -> CRCW06030000Z0EA
Changed lines of the file:
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@@
+			)
+		)
+		(property "PN" "CRCW06032K20FKEA"
+			(at 114.3 85.09 0)
+			(effects
+				(font
+					(size 1.27 1.27)
+				)
+				(hide yes)
 			)
 		)
@@
 			)
 		)
+		(property "PN" "SJ1-3523N"
+			(at 96.52 97.79 0)
+			(effects
+				(font
+					(size 1.27 1.27)
+				)
+				(hide yes)
+			)
+		)
 		(pin "S"
 		)
@@
 			)
 		)
+		(property "PN" "CRCW06030000Z0EA"
+			(at 105.41 111.76 0)
+			(effects
+				(font
+					(size 1.27 1.27)
+				)
+				(hide yes)
+			)
+		)
 		(pin "2"
 		)
@@
 		)
 		(instances
-			(project "nucleo_tdm_breakout1"
+			(project "tdm_b1"
 				(path "/c8dcc663-46e4-4dea-a66e-b8b88fdce1bb/ee5e271c-80f2-40af-99c0-532292736c08"
 					(page "7")
