File: tdm_b1/tdm_b1.kicad_sch (KiCad schematic)
At the start: 20 parts, among them J1 Conn_02x17_Odd_Even, J8 Conn_02x08_Odd_Even, J9 Conn_02x15_Odd_Even

Commit message: filled out part number for tdm_b1
Parts:
- C27: PN (none) -> GCM188R71C105KA64J
- C29, C30: PN (none) -> GCJ188R71H104KA12D
- J1: PN (none) -> PRPC017DAAN-RC
- J8: PN (none) -> 10129381-916001BLF
- J9: PN (none) -> PRPC015DAAN-RC
- R34, R37: PN (none) -> CRCW06030000Z0EA
Changed lines of the file:
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@@
+			)
+		)
+		(property "PN" "GCM188R71C105KA64J"
+			(at 137.16 59.69 0)
+			(effects
+				(font
+					(size 1.27 1.27)
+				)
+				(hide yes)
 			)
 		)
@@
 			)
 		)
+		(property "PN" "GCJ188R71H104KA12D"
+			(at 162.56 59.69 0)
+			(effects
+				(font
+					(size 1.27 1.27)
+				)
+				(hide yes)
+			)
+		)
 		(pin "1"
 		)
@@
 			)
 		)
+		(property "PN" "PRPC015DAAN-RC"
+			(at 91.44 110.49 0)
+			(effects
+				(font
+					(size 1.27 1.27)
+				)
+				(hide yes)
+			)
+		)
 		(pin "11"
 		)
@@
 			)
 		)
+		(property "PN" "CRCW06030000Z0EA"
+			(at 162.56 166.37 90)
+			(effects
+				(font
+					(size 1.27 1.27)
+				)
+				(hide yes)
+			)
+		)
 		(pin "2"
 		)
@@
 			)
 		)
+		(property "PN" "10129381-916001BLF"
+			(at 91.44 62.23 0)
+			(effects
+				(font
+					(size 1.27 1.27)
+				)
+				(hide yes)
+			)
+		)
 		(pin "9"
 		)
@@
 			)
 		)
+		(property "PN" "CRCW06030000Z0EA"
+			(at 163.83 176.53 90)
+			(effects
+				(font
+					(size 1.27 1.27)
+				)
+				(hide yes)
+			)
+		)
 		(pin "2"
 		)
@@
 			)
 		)
+		(property "PN" "GCJ188R71H104KA12D"
+			(at 149.86 59.69 0)
+			(effects
+				(font
+					(size 1.27 1.27)
+				)
+				(hide yes)
+			)
+		)
 		(pin "1"
 		)
@@
 		)
 		(property "Description" "Generic connector, double row, 02x17, odd/even pin numbering scheme (row 1 odd numbers, row 2 even numbers), script generated (kicad-library-utils/schlib/autogen/connector/)"
+			(at 185.42 109.22 0)
+			(effects
+				(font
+					(size 1.27 1.27)
+				)
+				(hide yes)
+			)
+		)
+		(property "PN" "PRPC017DAAN-RC"
 			(at 185.42 109.22 0)
 			(effects
@@
 		)
 		(instances
-			(project "nucleo_tdm_breakout1"
+			(project "tdm_b1"
 				(path "/c8dcc663-46e4-4dea-a66e-b8b88fdce1bb"
 					(page "4")
@@
 		)
 		(instances
-			(project "nucleo_tdm_breakout1"
+			(project "tdm_b1"
 				(path "/c8dcc663-46e4-4dea-a66e-b8b88fdce1bb"
 					(page "2")
@@
 		)
 		(instances
-			(project "nucleo_tdm_breakout1"
+			(project "tdm_b1"
 				(path "/c8dcc663-46e4-4dea-a66e-b8b88fdce1bb"
 					(page "10")
@@
 		)
 		(instances
-			(project "nucleo_tdm_breakout1"
+			(project "tdm_b1"
 				(path "/c8dcc663-46e4-4dea-a66e-b8b88fdce1bb"
 					(page "3")
@@
 		)
 		(instances
-			(project "nucleo_tdm_breakout1"
+			(project "tdm_b1"
 				(path "/c8dcc663-46e4-4dea-a66e-b8b88fdce1bb"
 					(page "8")
@@
 		)
 		(instances
-			(project "nucleo_tdm_breakout1"
+			(project "tdm_b1"
 				(path "/c8dcc663-46e4-4dea-a66e-b8b88fdce1bb"
 					(page "5")
@@
 		)
 		(instances
-			(project "nucleo_tdm_breakout1"
+			(project "tdm_b1"
 				(path "/c8dcc663-46e4-4dea-a66e-b8b88fdce1bb"
 					(page "6")
@@
 		)
 		(instances
-			(project "nucleo_tdm_breakout1"
+			(project "tdm_b1"
 				(path "/c8dcc663-46e4-4dea-a66e-b8b88fdce1bb"
 					(page "9")
@@
 		)
 		(instances
-			(project "nucleo_tdm_breakout1"
+			(project "tdm_b1"
 				(path "/c8dcc663-46e4-4dea-a66e-b8b88fdce1bb"
 					(page "11")
